Commit message: added new rb1 base, old version renamed to v0

File: rb1_base_description/robots/rb1_base_platform.urdf.xacro (robot description, xacro)
@@ -8,8 +8,9 @@
     <xacro:include filename="$(find rb1_base_description)/urdf/bases/rb1_base.urdf.xacro" />
 	<!-- Import RB1 wheels -->
-	<xacro:include filename="$(find rb1_base_description)/urdf/wheels/rubber_wheel.urdf.xacro" />
+	<xacro:include filename="$(find rb1_base_description)/urdf/wheels/rubber_wheel_.urdf.xacro" />
 	<xacro:include filename="$(find rb1_base_description)/urdf/wheels/omni_wheel.urdf.xacro" />
 	<!-- Import all available sensors -->
-	<xacro:include filename="$(find rb1_base_description)/urdf/sensors/all_sensors.urdf.xacro" />
+	<!-- xacro:include filename="$(find rb1_base_description)/urdf/sensors/all_sensors.urdf.xacro" / -->
+	<xacro:include filename="$(find robotnik_sensors)/urdf/all_sensors.urdf.xacro" />
 	<!-- ***************** -->
 	<!-- Global parameters -->
@@ -18,15 +19,13 @@
 	<!-- Wheel parameters -->
 	<xacro:property name="wheel_offset_x" value="0.0" />    <!-- x,y,z in translation from base_link to the center of the wheel -->
-	<xacro:property name="wheel_offset_y" value="0.183" />
+	<xacro:property name="wheel_offset_y" value="0.217" />
 	<xacro:property name="wheel_offset_z" value="0.051" />
 	<!-- Castor paramters -->
-	<xacro:property name="omni_back_x" value="0.185" />
+	<xacro:property name="omni_back_x" value="0.195" />
 	<xacro:property name="omni_back_y" value="0.0" />
-	<!-- xacro:property name="omni_back_z" value="0.028" / -->
-	<xacro:property name="omni_back_z" value="0.0265" />
+	<xacro:property name="omni_back_z" value="0.026" />
 	<xacro:property name="omni_front_x" value="0.133" />
-	<xacro:property name="omni_front_y" value="0.142" />
-	<!-- xacro:property name="omni_front_z" value="0.028" / -->
-	<xacro:property name="omni_front_z" value="0.0265" />
+	<xacro:property name="omni_front_y" value="0.144" />
+	<xacro:property name="omni_front_z" value="0.026" />
 	<!-- Flag to select the high or low quality model -->
 	<xacro:property name="hq" value="true" />
@@ -62,7 +61,10 @@
 		<origin xyz="0.210 0.0 0.305" rpy="0 0 0"/>
 	</xacro:sensor_hokuyo_utm30lx -->
-        <xacro:sensor_hokuyo_urg04lx name="hokuyo" parent="base_link">
-           <origin xyz="0.220 0.0 0.170" rpy="0 3.1416 3.1416"/>
-        </xacro:sensor_hokuyo_urg04lx>
+    <!-- xacro:sensor_hokuyo_urg04lx name="hokuyo" parent="base_link">
+        <origin xyz="0.223 0.0 0.209" rpy="0 3.1416 3.1416"/>
+    </xacro:sensor_hokuyo_urg04lx -->
+	<xacro:sensor_hokuyo_ust10lx name="hokuyo" parent="base_link">
+		<origin xyz="0.223 0.0 0.159" rpy="0 0 0"/>
+	</xacro:sensor_hokuyo_ust10lx>
 	<xacro:sensor_imu name="imu" parent="base_link">
 		<origin xyz="-0.18 0.0 0.170" rpy="0 0 0"/>

File: rb1_base_description/robots/rb1_base_platform_v0.urdf.xacro (robot description, xacro)
@@ -6,18 +6,10 @@
 	<!-- First we import all posible elements defined in the urdf.xacro files. All these elements are defined as macro:xacros -->
 	<!-- Import RB1 base elements -->
-    <xacro:include filename="$(find rb1_base_description)/urdf/bases/rb1_base.urdf.xacro" />
-    <gazebo>
-      <plugin name="ros_control" filename="libgazebo_ros_control.so">
-        <robotNamespace>/rb1</robotNamespace>
-        <robotParam>robot_description</robotParam>
-        <controlPeriod>0.001</controlPeriod>
-	    <robotSimType>gazebo_ros_control/DefaultRobotHWSim</robotSimType>
-      </plugin>
-    </gazebo>
+    <xacro:include filename="$(find rb1_base_description)/urdf/bases/rb1_base_v0.urdf.xacro" />
 	<!-- Import RB1 wheels -->
 	<xacro:include filename="$(find rb1_base_description)/urdf/wheels/rubber_wheel.urdf.xacro" />
 	<xacro:include filename="$(find rb1_base_description)/urdf/wheels/omni_wheel.urdf.xacro" />
 	<!-- Import all available sensors -->
-    <xacro:include filename="$(find robotnik_sensors)/urdf/all_sensors.urdf.xacro"/>
+	<xacro:include filename="$(find rb1_base_description)/urdf/sensors/all_sensors.urdf.xacro" />
 	<!-- ***************** -->
 	<!-- Global parameters -->
@@ -26,13 +18,13 @@
 	<!-- Wheel parameters -->
 	<xacro:property name="wheel_offset_x" value="0.0" />    <!-- x,y,z in translation from base_link to the center of the wheel -->
-	<xacro:property name="wheel_offset_y" value="0.217" />
+	<xacro:property name="wheel_offset_y" value="0.183" />
 	<xacro:property name="wheel_offset_z" value="0.051" />
 	<!-- Castor paramters -->
-	<xacro:property name="omni_back_x" value="0.195" />
+	<xacro:property name="omni_back_x" value="0.185" />
 	<xacro:property name="omni_back_y" value="0.0" />
-	<xacro:property name="omni_back_z" value="0.026" />
+	<xacro:property name="omni_back_z" value="0.0265" />
 	<xacro:property name="omni_front_x" value="0.133" />
-	<xacro:property name="omni_front_y" value="0.144" />
-	<xacro:property name="omni_front_z" value="0.026" />
+	<xacro:property name="omni_front_y" value="0.142" />
+	<xacro:property name="omni_front_z" value="0.0265" />
 	<!-- Flag to select the high or low quality model -->
 	<xacro:property name="hq" value="true" />
@@ -68,11 +60,7 @@
 		<origin xyz="0.210 0.0 0.305" rpy="0 0 0"/>
 	</xacro:sensor_hokuyo_utm30lx -->
-    <!-- xacro:sensor_hokuyo_urg04lx name="hokuyo1" parent="base_link">
-        <origin xyz="0.220 0.0 0.170" rpy="0 3.1416 3.1416"/>
-    </xacro:sensor_hokuyo_urg04lx -->
-	<xacro:sensor_hokuyo_ust10lx name="hokuyo" parent="base_link">
-		<!-- origin xyz="0.223 0.0 0.209" rpy="0 0 0"/ -->
-		<origin xyz="0.223 0.0 0.159" rpy="0 0 0"/>
-	</xacro:sensor_hokuyo_ust10lx>
+        <xacro:sensor_hokuyo_urg04lx name="hokuyo" parent="base_link">
+           <origin xyz="0.220 0.0 0.170" rpy="0 3.1416 3.1416"/>
+        </xacro:sensor_hokuyo_urg04lx>
 	<xacro:sensor_imu name="imu" parent="base_link">
 		<origin xyz="-0.18 0.0 0.170" rpy="0 0 0"/>

File: rb1_base_description/robots/rb1_base_platform_v0_standalone.urdf.xacro (robot description, xacro)
@@ -6,5 +6,5 @@
 	<!-- First we import all posible elements defined in the urdf.xacro files. All these elements are defined as macro:xacros -->
 	<!-- Import RB1 base elements -->
-    <xacro:include filename="$(find rb1_base_description)/urdf/bases/rb1_base.urdf.xacro" />
+    <xacro:include filename="$(find rb1_base_description)/urdf/bases/rb1_base_v0.urdf.xacro" />
     <gazebo>
       <plugin name="ros_control" filename="libgazebo_ros_control.so">
@@ -19,5 +19,6 @@
 	<xacro:include filename="$(find rb1_base_description)/urdf/wheels/omni_wheel.urdf.xacro" />
 	<!-- Import all available sensors -->
-    <xacro:include filename="$(find robotnik_sensors)/urdf/all_sensors.urdf.xacro"/>
+	<!-- xacro:include filename="$(find rb1_base_description)/urdf/sensors/all_sensors.urdf.xacro" / -->
+        <xacro:include filename="$(find robotnik_sensors)/urdf/all_sensors.urdf.xacro"/>
 	<!-- ***************** -->
 	<!-- Global parameters -->
@@ -26,13 +27,13 @@
 	<!-- Wheel parameters -->
 	<xacro:property name="wheel_offset_x" value="0.0" />    <!-- x,y,z in translation from base_link to the center of the wheel -->
-	<xacro:property name="wheel_offset_y" value="0.217" />
+	<xacro:property name="wheel_offset_y" value="0.183" />
 	<xacro:property name="wheel_offset_z" value="0.051" />
 	<!-- Castor paramters -->
-	<xacro:property name="omni_back_x" value="0.195" />
+	<xacro:property name="omni_back_x" value="0.185" />
 	<xacro:property name="omni_back_y" value="0.0" />
-	<xacro:property name="omni_back_z" value="0.026" />
+	<xacro:property name="omni_back_z" value="0.0265" />
 	<xacro:property name="omni_front_x" value="0.133" />
-	<xacro:property name="omni_front_y" value="0.144" />
-	<xacro:property name="omni_front_z" value="0.026" />
+	<xacro:property name="omni_front_y" value="0.142" />
+	<xacro:property name="omni_front_z" value="0.0265" />
 	<!-- Flag to select the high or low quality model -->
 	<xacro:property name="hq" value="true" />
@@ -65,14 +66,10 @@
 	</xacro:omni_wheel>
 	<!-- SENSORS -->
-	<!-- xacro:sensor_hokuyo_utm30lx name="hokuyo" parent="base_link">
+	<xacro:sensor_hokuyo_utm30lx name="hokuyo" parent="base_link">
 		<origin xyz="0.210 0.0 0.305" rpy="0 0 0"/>
-	</xacro:sensor_hokuyo_utm30lx -->
+	</xacro:sensor_hokuyo_utm30lx>
     <!-- xacro:sensor_hokuyo_urg04lx name="hokuyo1" parent="base_link">
         <origin xyz="0.220 0.0 0.170" rpy="0 3.1416 3.1416"/>
     </xacro:sensor_hokuyo_urg04lx -->
-	<xacro:sensor_hokuyo_ust10lx name="hokuyo" parent="base_link">
-		<!-- origin xyz="0.223 0.0 0.209" rpy="0 0 0"/ -->
-		<origin xyz="0.223 0.0 0.159" rpy="0 0 0"/>
-	</xacro:sensor_hokuyo_ust10lx>
 	<xacro:sensor_imu name="imu" parent="base_link">
 		<origin xyz="-0.18 0.0 0.170" rpy="0 0 0"/>

File: rb1_base_description/urdf/bases/rb1_base.gazebo.xacro (robot description, xacro)
@@ -2,5 +2,5 @@
 <robot xmlns:xacro="http://ros.org/wiki/xacro">
   <!-- ros control plugin -->
-  <xacro:macro name="ros_control">
+  <!-- xacro:macro name="ros_control">
     <gazebo>
       <plugin name="ros_control" filename="libgazebo_ros_control.so">
@@ -11,5 +11,5 @@
       </plugin>
     </gazebo>
-	</xacro:macro>
+	</xacro:macro -->
 	<!-- differential drive plugin -->
 	<xacro:macro name="diff_drive">

File: rb1_base_description/urdf/bases/rb1_base_v0.urdf.xacro (robot description, xacro)
@@ -33,10 +33,10 @@
        <xacro:if value="${hq}">
        <geometry>
-	     <mesh filename="package://rb1_base_description/meshes/bases/rb1_base.dae"/>
+	     <mesh filename="package://rb1_base_description/meshes/bases/rb1_base_v0.dae"/>
        </geometry>
        </xacro:if>
        <xacro:unless value="${hq}">
        <geometry>
-       <mesh filename="package://rb1_base_description/meshes/bases/rb1_base.stl"/>
+       <mesh filename="package://rb1_base_description/meshes/bases/rb1_base_v0.stl"/>
        </geometry>
        </xacro:unless>
@@ -48,5 +48,5 @@
        <origin xyz="0 0 0" rpy="0 0 0 " />
        <geometry>
-         <mesh filename="package://rb1_base_description/meshes/bases/rb1_base.dae"/>
+         <mesh filename="package://rb1_base_description/meshes/bases/rb1_base_v0.dae"/>
        </geometry>
     </collision>

Commit message: new model working in gazebo

File: rb1_base_description/robots/rb1_base_platform.urdf.xacro (robot description, xacro)
@@ -24,8 +24,8 @@
 	<xacro:property name="omni_back_x" value="0.195" />
 	<xacro:property name="omni_back_y" value="0.0" />
-	<xacro:property name="omni_back_z" value="0.026" />
+	<xacro:property name="omni_back_z" value="0.0265" />
 	<xacro:property name="omni_front_x" value="0.133" />
 	<xacro:property name="omni_front_y" value="0.144" />
-	<xacro:property name="omni_front_z" value="0.026" />
+	<xacro:property name="omni_front_z" value="0.0265" />
 	<!-- Flag to select the high or low quality model -->
 	<xacro:property name="hq" value="true" />

File: rb1_base_description/robots/rb1_base_platform_standalone.urdf.xacro (robot description, xacro)
@@ -31,8 +31,8 @@
 	<xacro:property name="omni_back_x" value="0.195" />
 	<xacro:property name="omni_back_y" value="0.0" />
-	<xacro:property name="omni_back_z" value="0.026" />
+	<xacro:property name="omni_back_z" value="0.0265" />
 	<xacro:property name="omni_front_x" value="0.133" />
 	<xacro:property name="omni_front_y" value="0.144" />
-	<xacro:property name="omni_front_z" value="0.026" />
+	<xacro:property name="omni_front_z" value="0.0265" />
 	<!-- Flag to select the high or low quality model -->
 	<xacro:property name="hq" value="true" />
@@ -72,5 +72,4 @@
     </xacro:sensor_hokuyo_urg04lx -->
 	<xacro:sensor_hokuyo_ust10lx name="hokuyo" parent="base_link">
-		<!-- origin xyz="0.223 0.0 0.209" rpy="0 0 0"/ -->
 		<origin xyz="0.223 0.0 0.159" rpy="0 0 0"/>
 	</xacro:sensor_hokuyo_ust10lx>

File: rb1_base_description/robots/rb1_base_platform_v0_standalone.urdf.xacro (robot description, xacro)
@@ -19,6 +19,5 @@
 	<xacro:include filename="$(find rb1_base_description)/urdf/wheels/omni_wheel.urdf.xacro" />
 	<!-- Import all available sensors -->
-	<!-- xacro:include filename="$(find rb1_base_description)/urdf/sensors/all_sensors.urdf.xacro" / -->
-        <xacro:include filename="$(find robotnik_sensors)/urdf/all_sensors.urdf.xacro"/>
+    <xacro:include filename="$(find robotnik_sensors)/urdf/all_sensors.urdf.xacro"/>
 	<!-- ***************** -->
 	<!-- Global parameters -->

Commit message: hokuyo upside down

File: rb1_base_description/robots/rb1_base_platform.urdf.xacro (robot description, xacro)
@@ -64,5 +64,5 @@
     </xacro:sensor_hokuyo_urg04lx -->
 	<xacro:sensor_hokuyo_ust10lx name="hokuyo" parent="base_link">
-		<origin xyz="0.223 0.0 0.159" rpy="0 0 0"/>
+		<origin xyz="0.223 0.0 0.159" rpy="0 3.1416 3.1416"/>
 	</xacro:sensor_hokuyo_ust10lx>
 	<xacro:sensor_imu name="imu" parent="base_link">

File: rb1_base_description/robots/rb1_base_platform_standalone.urdf.xacro (robot description, xacro)
@@ -71,6 +71,9 @@
         <origin xyz="0.220 0.0 0.170" rpy="0 3.1416 3.1416"/>
     </xacro:sensor_hokuyo_urg04lx -->
+	<!-- xacro:sensor_hokuyo_ust10lx name="hokuyo" parent="base_link">
+		<origin xyz="0.223 0.0 0.159" rpy="0 0 0"/>
+	</xacro:sensor_hokuyo_ust10lx -->
 	<xacro:sensor_hokuyo_ust10lx name="hokuyo" parent="base_link">
-		<origin xyz="0.223 0.0 0.159" rpy="0 0 0"/>
+		<origin xyz="0.223 0.0 0.159" rpy="0 3.1416 3.1416"/>
 	</xacro:sensor_hokuyo_ust10lx>
 	<xacro:sensor_imu name="imu" parent="base_link">
