Commit message: updated inertia parameters

File: rb1_base_description/urdf/bases/rb1_base.urdf.xacro (robot description, xacro)
@@ -27,5 +27,5 @@
       <mass value="25.0" />
       <origin xyz="0 0 0" />
-      <inertia  ixx="1.0" ixy="0.0"  ixz="0.0"  iyy="1.0"  iyz="0.0"  izz="1.0" />
+      <inertia  ixx="0.007" ixy="0.0"  ixz="0.0"  iyy="0.007"  iyz="0.0"  izz="0.78" />
     </inertial>
     <visual>
