Commit message: changes to clean error: no valid hardware interface element found in joint

File: rb1_arm_description/urdf/arms/rb1_arm_7dof.urdf.xacro (robot description, xacro)
@@ -1,5 +1,5 @@
 <?xml version="1.0"?>
 <robot name="rb1_arm_7dof" xmlns:xacro="http://www.ros.org/wiki/xacro">
-	<xacro:include filename="$(find rb1_arm_description)/urdf/arms/rb1_arm_7dof.gazebo.xacro" />
+	<!-- xacro:include filename="$(find rb1_arm_description)/urdf/arms/rb1_arm_7dof.gazebo.xacro" / -->
 	<xacro:property name="j1_mechanical_reduction" value="502.0"/>
 	<xacro:property name="j1_motor_torque_constant" value="50.0"/>
@@ -217,7 +217,9 @@
     <transmission name="j1_trans">
 	 <type>transmission_interface/SimpleTransmission</type>
-     <joint name="j1" />
+	 <joint name="j1">
+         <hardwareInterface>EffortJointInterface</hardwareInterface>
+     </joint>
      <actuator name="j1_motor">
-	    <hardwareInterface>EffortJointInterface</hardwareInterface>
+	    <!-- hardwareInterface>EffortJointInterface</hardwareInterface -->
         <mechanicalReduction>${j1_mechanical_reduction}</mechanicalReduction>
 		<motorTorqueConstant>${j1_motor_torque_constant}</motorTorqueConstant>
@@ -313,7 +315,8 @@
     <transmission name="j2_trans">
 	 <type>transmission_interface/SimpleTransmission</type>
-     <joint name="j2" />
+     <joint name="j2">
+		 <hardwareInterface>EffortJointInterface</hardwareInterface>
+     </joint>
      <actuator name="j2_motor">
-	    <hardwareInterface>EffortJointInterface</hardwareInterface>
         <mechanicalReduction>${j2_mechanical_reduction}</mechanicalReduction>
 		<motorTorqueConstant>${j2_motor_torque_constant}</motorTorqueConstant>
@@ -406,7 +409,8 @@
     <transmission name="j3_trans">
 	 <type>transmission_interface/SimpleTransmission</type>
-     <joint name="j3" />
+     <joint name="j3">
+		<hardwareInterface>EffortJointInterface</hardwareInterface>
+	 </joint>
      <actuator name="j3_motor">
-	    <hardwareInterface>EffortJointInterface</hardwareInterface>
         <mechanicalReduction>${j3_mechanical_reduction}</mechanicalReduction>
 		<motorTorqueConstant>${j3_motor_torque_constant}</motorTorqueConstant>
@@ -501,7 +505,8 @@
     <transmission name="j4_trans">
 	 <type>transmission_interface/SimpleTransmission</type>
-     <joint name="j4" />
+     <joint name="j4">
+        <hardwareInterface>EffortJointInterface</hardwareInterface>
+     </joint>
      <actuator name="j4_motor">
-	    <hardwareInterface>EffortJointInterface</hardwareInterface>
         <mechanicalReduction>${j4_mechanical_reduction}</mechanicalReduction>
 		<motorTorqueConstant>${j4_motor_torque_constant}</motorTorqueConstant>
@@ -594,7 +599,8 @@
     <transmission name="j5_trans">
 	 <type>transmission_interface/SimpleTransmission</type>
-     <joint name="j5" />
+     <joint name="j5">
+        <hardwareInterface>EffortJointInterface</hardwareInterface>
+     </joint>
      <actuator name="j5_motor">
-	    <hardwareInterface>EffortJointInterface</hardwareInterface>
         <mechanicalReduction>${j5_mechanical_reduction}</mechanicalReduction>
 		<motorTorqueConstant>${j5_motor_torque_constant}</motorTorqueConstant>
@@ -689,7 +695,8 @@
     <transmission name="j6_trans">
 	 <type>transmission_interface/SimpleTransmission</type>
-     <joint name="j6" />
+     <joint name="j6">
+		<hardwareInterface>EffortJointInterface</hardwareInterface>
+	 </joint>
      <actuator name="j6_motor">
-	    <hardwareInterface>EffortJointInterface</hardwareInterface>
         <mechanicalReduction>${j6_mechanical_reduction}</mechanicalReduction>
 		<motorTorqueConstant>${j6_motor_torque_constant}</motorTorqueConstant>
@@ -709,7 +716,8 @@
     <transmission name="j7_trans">
 		<type>transmission_interface/SimpleTransmission</type>
-		<joint name="j7" />
+		<joint name="j7">
+			<hardwareInterface>EffortJointInterface</hardwareInterface>
+		</joint>
 		<actuator name="j7_motor">
-			<hardwareInterface>EffortJointInterface</hardwareInterface>
 			<mechanicalReduction>${j7_mechanical_reduction}</mechanicalReduction>
 			<motorTorqueConstant>${j7_motor_torque_constant}</motorTorqueConstant>

File: rb1_arm_description/urdf/grippers/rb1_gripper_1.urdf.xacro (robot description, xacro)
@@ -157,7 +157,8 @@
   <transmission name="jg2_trans">
 	 <type>transmission_interface/SimpleTransmission</type>
-     <joint name="jg2" />
+     <joint name="jg2">
+        <hardwareInterface>EffortJointInterface</hardwareInterface>
+     </joint>
      <actuator name="jg2_motor">
-	    <hardwareInterface>EffortJointInterface</hardwareInterface>
         <mechanicalReduction>${finger_mechanical_reduction}</mechanicalReduction>
 		<motorTorqueConstant>${finger_motor_torque_constant}</motorTorqueConstant>

File: rb1_arm_description/urdf/grippers/two_finger_gripper.urdf.xacro (robot description, xacro)
@@ -106,7 +106,8 @@
   <transmission name="jg1_trans">
 	 <type>transmission_interface/SimpleTransmission</type>
-     <joint name="jg1" />
+     <joint name="jg1">
+		<hardwareInterface>EffortJointInterface</hardwareInterface>
+	 </joint>
      <actuator name="jg1_motor">
-	    <hardwareInterface>EffortJointInterface</hardwareInterface>
         <mechanicalReduction>${finger_mechanical_reduction}</mechanicalReduction>
 		<motorTorqueConstant>${finger_motor_torque_constant}</motorTorqueConstant>
@@ -170,7 +171,8 @@
   <transmission name="jg2_trans">
 	 <type>transmission_interface/SimpleTransmission</type>
-     <joint name="jg2" />
+     <joint name="jg2">
+		 <hardwareInterface>EffortJointInterface</hardwareInterface>
+     </joint>
      <actuator name="jg2_motor">
-	    <hardwareInterface>EffortJointInterface</hardwareInterface>
         <mechanicalReduction>${finger_mechanical_reduction}</mechanicalReduction>
 		<motorTorqueConstant>${finger_motor_torque_constant}</motorTorqueConstant>

File: rb1_base_description/urdf/bases/rb1_base.gazebo.xacro (robot description, xacro)
@@ -2,5 +2,5 @@
 <robot xmlns:xacro="http://ros.org/wiki/xacro">
   <!-- ros control plugin -->
-  <!-- xacro:macro name="ros_control">
+  <xacro:macro name="ros_control">
     <gazebo>
       <plugin name="ros_control" filename="libgazebo_ros_control.so">
@@ -11,5 +11,5 @@
       </plugin>
     </gazebo>
-	</xacro:macro -->
+	</xacro:macro>
 	<!-- differential drive plugin -->
 	<xacro:macro name="diff_drive">

File: rb1_base_description/urdf/sensors/kinect.urdf.xacro (robot description, xacro)
@@ -125,4 +125,5 @@
           <distortion_t2>0.0</distortion_t2>
           <pointCloudCutoff>0.4</pointCloudCutoff>
+          <pointCloudCutoffMax>5.0</pointCloudCutoffMax>
         </plugin>
       </sensor>

File: rb1_base_description/urdf/wheels/rubber_wheel.urdf.xacro (robot description, xacro)
@@ -58,8 +58,11 @@
     <transmission name="${name}_wheel_joint_trans">
       <type>transmission_interface/SimpleTransmission</type>
-      <joint name="joint_${name}_wheel" />
+      <joint name="joint_${name}_wheel">
+          <hardwareInterface>EffortJointInterface</hardwareInterface>
+      </joint>
       <actuator name="${name}_wheel_joint_motor">
-        <hardwareInterface>EffortJointInterface</hardwareInterface>
+        <!-- hardwareInterface>EffortJointInterface</hardwareInterface -->
         <mechanicalReduction>1</mechanicalReduction>
+        <motorTorqueConstant>10</motorTorqueConstant>
       </actuator>
     </transmission>

File: rb1_description/robots/rb1_robot.urdf (robot description, URDF)
Before this commit: robot rb1, 38 links, 37 joints
Joints:
- joint j1: limit lower=-1.570796327 upper=1.570796327 effort=60.0 velocity=2.9217 -> lower=-1.55 upper=1.55 effort=60.0 velocity=2.9217
- joint j2: limit lower=-1.570796327 upper=1.570796327 effort=60.0 velocity=2.9217 -> lower=-1.95 upper=1.55 effort=60.0 velocity=2.9217
- joint j4: limit lower=-1.570796327 upper=1.570796327 effort=35.0 velocity=3.1527 -> lower=-1.95 upper=1.95 effort=35.0 velocity=3.1527
- joint j6: limit lower=-1.570796327 upper=1.570796327 effort=8.0 velocity=2.98452 -> lower=-1.57 upper=1.57 effort=8.0 velocity=2.98452

File: rb1_description/robots/rb1_robot.urdf.xacro (robot description, xacro)
@@ -13,5 +13,5 @@
 	<!-- Gazebo ros control plugins -->
 	<!-- xacro:ros_control/ -->
-    <gazebo>
+    <!-- gazebo>
       <plugin name="ros_control" filename="libgazebo_ros_control.so">
         <robotNamespace>/rb1</robotNamespace>
@@ -20,5 +20,5 @@
 	    <robotSimType>gazebo_ros_control/DefaultRobotHWSim</robotSimType>
       </plugin>
-    </gazebo>
+    </gazebo -->
 	<!-- Fix torso to base -->
 	<joint

File: rb1_torso_description/urdf/rb1_torso_3dof.urdf.xacro (robot description, xacro)
@@ -106,7 +106,8 @@
   <transmission name="j1_torso_trans">
 	 <type>transmission_interface/SimpleTransmission</type>
-     <joint name="j1_torso" />
+     <joint name="j1_torso">
+		 <hardwareInterface>EffortJointInterface</hardwareInterface>
+     </joint>
      <actuator name="j1_torso_motor">
-	    <hardwareInterface>EffortJointInterface</hardwareInterface>
         <mechanicalReduction>${j1_torso_mechanical_reduction}</mechanicalReduction>
 		<motorTorqueConstant>${j1_torso_motor_torque_constant}</motorTorqueConstant>
@@ -156,7 +157,8 @@
   <transmission name="j1_head_trans">
 	 <type>transmission_interface/SimpleTransmission</type>
-     <joint name="j1_head" />
+     <joint name="j1_head">
+        <hardwareInterface>EffortJointInterface</hardwareInterface>
+     </joint>
      <actuator name="j1_head_motor">
-	    <hardwareInterface>EffortJointInterface</hardwareInterface>
         <mechanicalReduction>${j1_head_mechanical_reduction}</mechanicalReduction>
 		<motorTorqueConstant>${j1_head_motor_torque_constant}</motorTorqueConstant>
@@ -208,7 +210,8 @@
   <transmission name="j2_head_trans">
 	 <type>transmission_interface/SimpleTransmission</type>
-     <joint name="j2_head" />
+     <joint name="j2_head">
+		<hardwareInterface>EffortJointInterface</hardwareInterface>
+	 </joint>
      <actuator name="j2_head_motor">
-	    <hardwareInterface>EffortJointInterface</hardwareInterface>
         <mechanicalReduction>${j2_head_mechanical_reduction}</mechanicalReduction>
 		<motorTorqueConstant>${j2_head_motor_torque_constant}</motorTorqueConstant>

Commit message: changed base link name

File: rb1_arm_description/urdf/arms/rb1_arm_7dof.urdf.xacro (robot description, xacro)
@@ -1,5 +1,4 @@
 <?xml version="1.0"?>
 <robot name="rb1_arm_7dof" xmlns:xacro="http://www.ros.org/wiki/xacro">
-	<!-- xacro:include filename="$(find rb1_arm_description)/urdf/arms/rb1_arm_7dof.gazebo.xacro" / -->
 	<xacro:property name="j1_mechanical_reduction" value="502.0"/>
 	<xacro:property name="j1_motor_torque_constant" value="50.0"/>
@@ -42,5 +41,5 @@
     <xacro:property name="PI" value="3.1415926535897931"/>
     <!-- BASE_LINK -->
-    <link
+    <!-- link
       name="base_link_rb1_arm">
     </link>
@@ -57,7 +56,8 @@
 		<axis
 		  xyz="0 0 0" />
-	</joint>
+	</joint -->
 	<!-- 01 -->
-	<link name="link01_rb1_arm">
+	<!-- link name="link01_rb1_arm" -->
+	<link name="base_link_rb1_arm">
 		<inertial>
 		  <mass value="0.506" />
@@ -124,6 +124,8 @@
 		  xyz="0.0 0.0 0.0"
 		  rpy="0.0 0.0 0.0" />
+		<!-- parent
+		  link="link01_rb1_arm" / -->
 		<parent
-		  link="link01_rb1_arm" />
+		  link="base_link_rb1_arm" />
 		<child
 		  link="motor01_rb1_arm" />
@@ -209,5 +211,6 @@
 			xyz="0 0 0"
 			rpy="0.0 0.0 0.0" />
-		<parent link="link01_rb1_arm" />
+		<!-- parent link="link01_rb1_arm" /-->
+		<parent link="base_link_rb1_arm" />
 		<child link="link12_rb1_arm" />
 		<axis xyz="0 0 1" />
@@ -497,6 +500,4 @@
 	  <parent link="link34_rb1_arm" />
       <child link="link45_rb1_arm" />
-      <!-- check -->
-      <!-- xis xyz="0 0 -1" / -->
       <axis xyz="0 0 1"/>
       <limit effort="${joint_effort_limit_H54_100}" velocity="${joint_velocity_limit_H54_100}" upper="${j4_upper_limit}" lower="${j4_lower_limit}"/>
@@ -687,6 +688,4 @@
 	  <parent link="link56_rb1_arm" />
       <child link="link67_rb1_arm" />
-      <!-- check -->
-      <!-- axis xyz="0 0 -1" / -->
       <axis xyz="0 0 1"/>
       <limit effort="${joint_effort_limit_L42}" velocity="${joint_velocity_limit_L42}" upper="${j6_upper_limit}" lower="${j6_lower_limit}"/>
