Commit message: urdf from last xacro, working

File: rb1_description/robots/rb1_robot.urdf (robot description, URDF)
Before this commit: robot rb1, 38 links, 37 joints
Links:
- removed link link01_rb1_arm
- link base_link_rb1_arm: mass None -> 0.506; geometry collision mesh filename=package://rb1_arm_description/meshes/arms/armRB1_1_link.dae; visual mesh filename=package://rb1_arm_description/meshes/arms/armRB1_1_link.dae
- link hokuyo_laser_link: geometry collision box size=0.1 0.1 0.08; visual mesh filename=package://robotnik_sensors/meshes/hokuyo_ust_10lx.dae
- link left_wheel: geometry collision cylinder length=0.025 radius=0.076; visual mesh filename=package://rb1_base_description/meshes/wheels/wheel_rubber_6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
- link right_wheel: geometry collision cylinder length=0.025 radius=0.076; visual mesh filename=package://rb1_base_description/meshes/wheels/wheel_rubber_6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
- link xtion_head_cam_link: geometry collision box size=0.0730 .2760 0.0720; visual mesh filename=package://robotnik_sensors/meshes/asus_xtion_pro_live.dae scale=0.001 0.001 0.001
Joints:
- removed joint j1_rb1_arm
- joint hokuyo_laser_joint: origin xyz=0.220 0.0 0.170 rpy=0 3.1416 3.1416 -> xyz=0.223 0.0 0.159 rpy=0 3.1416 3.1416
- joint j01m_rb1_arm: parent link01_rb1_arm -> base_link_rb1_arm
- joint j1: parent link01_rb1_arm -> base_link_rb1_arm
- joint joint_left_wheel: origin xyz=0.0 0.183 0.051 rpy=0 0 0 -> xyz=0.0 0.217 0.051 rpy=0 0 0
- joint joint_omni_back_wheel: origin xyz=-0.185 0.0 0.0265 rpy=0 0 0 -> xyz=-0.195 0.0 0.0265 rpy=0 0 0
- joint joint_omni_front_left_wheel: origin xyz=0.133 0.142 0.0265 rpy=0 0 0 -> xyz=0.133 0.144 0.0265 rpy=0 0 0
- joint joint_omni_front_right_wheel: origin xyz=0.133 -0.142 0.0265 rpy=0 0 0 -> xyz=0.133 -0.144 0.0265 rpy=0 0 0
- joint joint_right_wheel: origin xyz=0.0 -0.183 0.051 rpy=0 0 0 -> xyz=0.0 -0.217 0.051 rpy=0 0 0
