Commit message: updated robot urdf for v2 version

File: rb1_description/robots/rb1_robot_mico_3fg_v0.urdf.xacro (robot description, xacro)
@@ -24,5 +24,5 @@
       type="fixed">
     <origin
-      xyz="-0.133 0.0 0.213"
+      xyz="0.0 0.0 0.0"
       rpy="0.0 0.0 0.0" />
     <parent
@@ -38,5 +38,5 @@
       type="fixed">
     <origin
-      xyz="0.055 0.0 0.0755"
+      xyz="0.074 0.0 0.668"
       rpy="0.0 0.0 0.0" />
     <parent

File: rb1_torso_description/robots/rb1_torso.urdf.xacro (robot description, xacro)
@@ -18,7 +18,11 @@
 	<xacro:rb1_torso_3dof name="rb1_torso_3dof" hq="${hq}" />
 	<!-- Ixtion sensor in head -->
-	<xacro:sensor_asus_xtion_pro name="xtion_head" parent="link2_head">
+	<!-- xacro:sensor_asus_xtion_pro name="xtion_head" parent="link2_head">
         <origin xyz="0.055 0.000 0.028" rpy="0 0 0"/>
-   </xacro:sensor_asus_xtion_pro>
+    </xacro:sensor_asus_xtion_pro -->
+    <!-- RGBD sensor -->
+    <xacro:sensor_orbbec_astra name="orbbec_astra_head" parent="link2_head">
+        <origin xyz="0.055 0.0125 0.028" rpy="0 0 0"/>
+    </xacro:sensor_orbbec_astra>
 	<!-- Gazebo ros control plugins -->
 	<!-- xacro:ros_control/ -->

File: rb1_torso_description/robots/rb1_torso_standalone.urdf.xacro (robot description, xacro)
@@ -22,5 +22,5 @@
         <origin xyz="0.055 0.000 0.028" rpy="0 0 0"/>
     </xacro:sensor_asus_xtion_pro -->
-    <xacro:sensor_orbbec_astra name="orbbec_astra" parent="link2_head">
+    <xacro:sensor_orbbec_astra name="orbbec_astra_head" parent="link2_head">
         <origin xyz="0.055 0.0125 0.028" rpy="0 0 0"/>
     </xacro:sensor_orbbec_astra>
