Commit message: moved arm 100 mm to front to avoid non-existant collision. Only solution will be changing stl :(

File: rb1_description/robots/rb1_robot_jaco_3fg.urdf (robot description, URDF)
Before this commit: robot rb1, 40 links, 39 joints
Joints:
- joint j_torso_arm: origin xyz=0.055 0.0 0.0755 rpy=0.0 0.0 0.0 -> xyz=0.155 0.0 0.0755 rpy=0.0 0.0 0.0

File: rb1_description/robots/rb1_robot_jaco_3fg.urdf.xacro (robot description, xacro)
@@ -38,6 +38,9 @@
 	  name="j_torso_arm"
       type="fixed">
+    <!-- origin
+      xyz="0.055 0.0 0.0755"
+      rpy="0.0 0.0 0.0" / -->
     <origin
-      xyz="0.055 0.0 0.0755"
+      xyz="0.155 0.0 0.0755"
       rpy="0.0 0.0 0.0" />
     <parent

Commit message: base set to old version

File: rb1_description/robots/rb1_robot_jaco_3fg.urdf (robot description, URDF)
Before this commit: robot rb1, 40 links, 39 joints
Links:
- removed link front_cover_link
- removed link orbbec_astra_cam_depth_frame
- removed link orbbec_astra_cam_depth_optical_frame
- removed link orbbec_astra_cam_link
- removed link orbbec_astra_cam_rgb_frame
- removed link orbbec_astra_cam_rgb_optical_frame
- link base_link: geometry collision mesh filename=package://rb1_base_description/meshes/bases/rb1_base_v0.dae; visual mesh filename=package://rb1_base_description/meshes/bases/rb1_base_v0.dae
- link hokuyo_laser_link: geometry collision box size=0.1 0.1 0.08; visual mesh filename=package://robotnik_sensors/meshes/hokuyo_urg_04lx.dae
Joints:
- removed joint front_cover_joint
- removed joint orbbec_astra_cam_depth_joint
- removed joint orbbec_astra_cam_depth_optical_joint
- removed joint orbbec_astra_cam_joint
- removed joint orbbec_astra_cam_rgb_joint
- removed joint orbbec_astra_cam_rgb_optical_joint
- joint hokuyo_laser_joint: origin xyz=0.223 0.0 0.159 rpy=0 3.1416 3.1416 -> xyz=0.220 0.0 0.170 rpy=0 3.1416 3.1416
- joint joint_left_wheel: origin xyz=0.0 0.217 0.051 rpy=0 0 0 -> xyz=0.0 0.183 0.051 rpy=0 0 0
- joint joint_omni_back_wheel: origin xyz=-0.195 0.0 0.0265 rpy=0 0 0 -> xyz=-0.185 0.0 0.0265 rpy=0 0 0
- joint joint_omni_front_left_wheel: origin xyz=0.133 0.148 0.0265 rpy=0 0 0 -> xyz=0.133 0.142 0.0265 rpy=0 0 0
- joint joint_omni_front_right_wheel: origin xyz=0.133 -0.148 0.0265 rpy=0 0 0 -> xyz=0.133 -0.142 0.0265 rpy=0 0 0
- joint joint_right_wheel: origin xyz=0.0 -0.217 0.051 rpy=0 0 0 -> xyz=0.0 -0.183 0.051 rpy=0 0 0

File: rb1_description/robots/rb1_robot_jaco_3fg.urdf.xacro (robot description, xacro)
@@ -12,5 +12,6 @@
 	<!-- First we import all posible elements defined in the urdf.xacro files. All these elements are defined as macro:xacros -->
 	<!-- Import RB1 base -->
-	<xacro:include filename="$(find rb1_base_description)/robots/rb1_base_platform.urdf.xacro" />
+	<!-- xacro:include filename="$(find rb1_base_description)/robots/rb1_base_platform.urdf.xacro" / -->
+        <xacro:include filename="$(find rb1_base_description)/robots/rb1_base_platform_v0.urdf.xacro" />
 	<!-- Import RB1 torso -->
 	<xacro:include filename="$(find rb1_torso_description)/robots/rb1_torso.urdf.xacro" />

Commit message: to dist 300 mm to test

File: rb1_description/robots/rb1_robot_jaco_3fg.urdf (robot description, URDF)
Before this commit: robot rb1, 34 links, 33 joints
Joints:
- joint j_torso_arm: origin xyz=0.155 0.0 0.0755 rpy=0.0 0.0 0.0 -> xyz=0.355 0.0 0.0755 rpy=0.0 0.0 0.0

File: rb1_description/robots/rb1_robot_jaco_3fg.urdf.xacro (robot description, xacro)
@@ -43,5 +43,5 @@
       rpy="0.0 0.0 0.0" / -->
     <origin
-      xyz="0.155 0.0 0.0755"
+      xyz="0.355 0.0 0.0755"
       rpy="0.0 0.0 0.0" />
     <parent

Commit message: temporary position to allow firmware home of kinova

File: rb1_description/robots/rb1_robot_jaco_3fg.urdf (robot description, URDF)
Before this commit: robot rb1, 34 links, 33 joints
Joints:
- joint j_torso_arm: origin xyz=0.355 0.0 0.0755 rpy=0.0 0.0 0.0 -> xyz=0.100 -0.315 0.1755 rpy=0.0 0.0 0.0

File: rb1_description/robots/rb1_robot_jaco_3fg.urdf.xacro (robot description, xacro)
@@ -35,4 +35,6 @@
       xyz="0 0 0" />
   </joint>
+  <!-- temporary offset - until home seq can be changed -->
+  <!-- 55 mm +X, 315 mm -Y, 100 mm +Z -->
   <!-- Fix arm to torso -->
   <joint
@@ -43,5 +45,5 @@
       rpy="0.0 0.0 0.0" / -->
     <origin
-      xyz="0.355 0.0 0.0755"
+      xyz="0.100 -0.315 0.1755"
       rpy="0.0 0.0 0.0" />
     <parent
