Commit message: rb1_description: updated rb1_jaco to new torso model

File: rb1_description/robots/rb1_robot_jaco_3fg_v3.urdf.xacro (robot description, xacro)
@@ -18,8 +18,8 @@
 	<xacro:include filename="$(find robotnik_sensors)/urdf/all_sensors.urdf.xacro" />
 	<!-- Import Jaco Arm -->
-	<xacro:include filename="$(find jaco_model)/urdf/jaco_arm.xacro" />
+	<xacro:include filename="$(find kinova_description)/urdf/j2n6s300.xacro" />
 	<!-- Fix torso to base -->
 	<joint
-	  name="j_base_torso"
+	  name="base_torso_joint"
       type="fixed">
     <origin
@@ -29,5 +29,5 @@
       link="base_link" />
     <child
-      link="base_link_rb1_torso" />
+      link="torso_base_link" />
     <axis
       xyz="0 0 0" />
@@ -35,5 +35,5 @@
   <!-- Fix arm to torso -->
   <joint
-	  name="j_torso_arm"
+	  name="torso_arm_joint"
       type="fixed">
     <!--origin
@@ -44,13 +44,13 @@
       rpy="0.0 0.0 0.0" />
     <parent
-      link="link2_torso" />
+      link="torso_slider_link" />
     <child
-      link="arm_link_base" />
+      link="torso_arm_link" />
     <axis
       xyz="0 0 0" />
   </joint>
-  <link name="arm_link_base" />
+   <link name="torso_arm_link" />
   <!-- arm -->
-  <xacro:jaco_arm parent="arm_link_base"/>
+  <xacro:j2n6s300 base_parent="torso_arm_link"/>
 	<!-- Gazebo ros control pluggins -->
 	<!-- xacro:ros_control/ -->

Commit message: rb1_description: added new torso

File: rb1_description/robots/rb1_robot_jaco_3fg_v3.urdf.xacro (robot description, xacro)
@@ -14,9 +14,12 @@
 	<xacro:include filename="$(find rb1_base_description)/robots/rb1_base_platform_v3.urdf.xacro" />
 	<!-- Import RB1 torso -->
-	<xacro:include filename="$(find rb1_torso_description)/robots/rb1_torso.urdf.xacro" />
+	<xacro:include filename="$(find rb1_torso_description)/urdf/rb1_torso_3dof_v3.urdf.xacro" />
 	<!-- Import all available sensors -->
 	<xacro:include filename="$(find robotnik_sensors)/urdf/all_sensors.urdf.xacro" />
 	<!-- Import Jaco Arm -->
 	<xacro:include filename="$(find kinova_description)/urdf/j2n6s300.xacro" />
+    <!-- base is added automatically when including xacro -->
+    <!-- add torso -->
+    <xacro:rb1_torso_3dof hq="false"/>
 	<!-- Fix torso to base -->
 	<joint
@@ -24,5 +27,5 @@
       type="fixed">
     <origin
-      xyz="-0.133 0.0 0.227"
+      xyz="0.0 0.0 0.223"
       rpy="0.0 0.0 0.0" />
     <parent
@@ -33,4 +36,9 @@
       xyz="0 0 0" />
   </joint>
+  <!-- add camera to head -->
+      <!-- RGBD sensor -->
+    <xacro:sensor_orbbec_astra name="head_camera" parent="head_tilt_link">
+        <origin xyz="0.055 0.0125 0.028" rpy="0 0 0"/>
+    </xacro:sensor_orbbec_astra>
   <!-- Fix arm to torso -->
   <joint
@@ -41,5 +49,5 @@
       rpy="0.0 0.0 0.0" / -->
     <origin
-      xyz="0.055 0.0 0.010"
+      xyz="0.0 0.0 0.075"
       rpy="0.0 0.0 0.0" />
     <parent

File: rb1_torso_description/urdf/rb1_torso_3dof_v3.urdf.xacro (robot description, xacro)
@@ -14,5 +14,5 @@
   <xacro:property name="head_tilt_joint_mechanical_reduction" value="320.0"/>
   <xacro:property name="head_tilt_joint_motor_torque_constant" value="1.0"/>
-  <xacro:macro name="rb1_torso_3dof" params="name hq">
+  <xacro:macro name="rb1_torso_3dof" params="hq">
   <!-- Robot mechanical and motor parameters -->
   <xacro:property name="PI" value="3.1415926535897931"/>

Commit message: rb1_description:jaco v3 model added

File: rb1_description/robots/rb1_robot_jaco_3fg_v3.urdf.xacro (robot description, xacro)
@@ -13,4 +13,5 @@
 	<!-- Import RB1 base -->
 	<xacro:include filename="$(find rb1_base_description)/robots/rb1_base_platform_v3.urdf.xacro" />
+	<xacro:include filename="$(find rb1_base_description)/urdf/others/tayg_box_6415.urdf.xacro" />
 	<!-- Import RB1 torso -->
 	<xacro:include filename="$(find rb1_torso_description)/robots/rb1_torso.urdf.xacro" />
@@ -53,4 +54,8 @@
   <!-- arm -->
   <xacro:j2n6s300 base_parent="torso_arm_link"/>
+  <!-- box -->
+  <xacro:tayg_box parent="top_cover_link" prefix="base_">
+      <origin xyz="0.175024 0 0" rpy="0 0 0" />
+  </xacro:tayg_box>
 	<!-- Gazebo ros control pluggins -->
 	<!-- xacro:ros_control/ -->

Commit message: rb1_description:rb1_torso description updated to new torso v3.

File: rb1_description/robots/rb1_robot_jaco_3fg_v3.urdf.xacro (robot description, xacro)
@@ -64,5 +64,5 @@
   <!-- box -->
   <xacro:tayg_box parent="top_cover_link" prefix="base_">
-      <origin xyz="0.175024 0 0" rpy="0 0 0" />
+	     <origin xyz="0.175024 0 0.003" rpy="0 0 0" />
   </xacro:tayg_box>
 	<!-- Gazebo ros control pluggins -->
