Commit message: updated rb1_robot_mico_3fg xacro

File: rb1_description/robots/rb1_robot_mico_3fg.urdf.xacro (robot description, xacro)
@@ -6,5 +6,5 @@
 	<xacro:property name="PI" value="3.1415926535897931"/>
 	<!-- Flag to select the high or low quality model -->
-	<xacro:property name="hq" value="true" />
+	<xacro:property name="hq" value="false" />
 	<!-- ***************** -->
 	<!-- Imported elements -->
@@ -37,6 +37,9 @@
 	  name="j_torso_arm"
       type="fixed">
+    <!--origin
+      xyz="0.055 0.0 0.0755"
+      rpy="0.0 0.0 0.0" / -->
     <origin
-      xyz="0.055 0.0 0.0755"
+      xyz="0.055 0.0 0.010"
       rpy="0.0 0.0 0.0" />
     <parent

Commit message: description: updated joint names of rb1_robot_mico

File: rb1_description/robots/rb1_robot_mico_3fg.urdf.xacro (robot description, xacro)
@@ -13,27 +13,37 @@
 	<!-- Import RB1 base -->
 	<xacro:include filename="$(find rb1_base_description)/robots/rb1_base_platform.urdf.xacro" />
+        <xacro:include filename="$(find rb1_base_description)/urdf/common.gazebo.xacro" />
 	<!-- Import RB1 torso -->
-	<xacro:include filename="$(find rb1_torso_description)/robots/rb1_torso.urdf.xacro" />
+	<xacro:include filename="$(find rb1_torso_description)/urdf/rb1_torso_3dof_v3.urdf.xacro" />
 	<!-- Import all available sensors -->
 	<xacro:include filename="$(find robotnik_sensors)/urdf/all_sensors.urdf.xacro" />
 	<!-- Import Mico Arm -->
-	<xacro:include filename="$(find mico_description)/robots/mico_arm_3fg_rb1.urdf.xacro" />
+	<!-- xacro:include filename="$(find mico_description)/robots/mico_arm_3fg_rb1.urdf.xacro" /-->
+	<!-- Import Jaco Arm -->
+	<xacro:include filename="$(find kinova_description)/urdf/m1n6s300.xacro" />
+    <!-- add torso -->
+    <xacro:rb1_torso_3dof hq="false"/>
 	<!-- Fix torso to base -->
 	<joint
-	  name="j_base_torso"
+	  name="base_torso_joint"
       type="fixed">
     <origin
-      xyz="-0.133 0.0 0.213"
+      xyz="0.0 0.0 0.223"
       rpy="0.0 0.0 0.0" />
     <parent
       link="base_link" />
     <child
-      link="base_link_rb1_torso" />
+      link="torso_base_link" />
     <axis
       xyz="0 0 0" />
   </joint>
+  <!-- add camera to head -->
+      <!-- RGBD sensor -->
+    <xacro:sensor_orbbec_astra prefix="head_camera" parent="head_tilt_link">
+        <origin xyz="0.055 0.0125 0.028" rpy="0 0 0"/>
+    </xacro:sensor_orbbec_astra>
   <!-- Fix arm to torso -->
   <joint
-	  name="j_torso_arm"
+	  name="torso_arm_joint"
       type="fixed">
     <!--origin
@@ -41,14 +51,17 @@
       rpy="0.0 0.0 0.0" / -->
     <origin
-      xyz="0.055 0.0 0.010"
+      xyz="0.0 0.0 0.075"
       rpy="0.0 0.0 0.0" />
     <parent
-      link="link2_torso" />
+      link="torso_slider_link" />
     <child
-      link="mico_link_base" />
+      link="torso_arm_link" />
     <axis
       xyz="0 0 0" />
   </joint>
+   <link name="torso_arm_link" />
+  <!-- arm -->
+  <xacro:m1n6s300 base_parent="torso_arm_link"/>
 	<!-- Gazebo ros control pluggins -->
-	<!-- xacro:ros_control/ -->
+	<xacro:ros_control/>
 </robot>
