Commit message: updated description - and will need some more...

File: rb1_description/robots/rb1_robot_jaco_3fg.urdf.xacro (robot description, xacro)
@@ -38,9 +38,6 @@
 	  name="j_torso_arm"
       type="fixed">
-    <!-- origin
+    <origin
       xyz="0.055 0.0 0.0755"
-      rpy="0.0 0.0 0.0" / -->
-    <origin
-      xyz="0.065 0.0 0.0755"
       rpy="0.0 0.0 0.0" />
     <parent
@@ -56,4 +53,4 @@
   <!-- xacro:ros_control/ -->
   <!-- arm -->
-  <xacro:jaco_arm  parent="arm_link_base"/>
+  <xacro:jaco_arm parent="arm_link_base"/>
 </robot>

Commit message: Update to kinetic

File: rb1_description/robots/rb1_robot_jaco_3fg.urdf.xacro (robot description, xacro)
@@ -13,5 +13,5 @@
 	<!-- Import RB1 base -->
 	<!-- xacro:include filename="$(find rb1_base_description)/robots/rb1_base_platform.urdf.xacro" / -->
-        <xacro:include filename="$(find rb1_base_description)/robots/rb1_base_platform_v0.urdf.xacro" />
+  	<xacro:include filename="$(find rb1_base_description)/robots/rb1_base_std.urdf.xacro" />
 	<!-- Import RB1 torso -->
 	<xacro:include filename="$(find rb1_torso_description)/robots/rb1_torso.urdf.xacro" />
@@ -20,43 +20,26 @@
 	<!-- Import Jaco Arm -->
 	<!-- xacro:include filename="$(find mico_description)/robots/mico_arm_3fg_rb1.urdf.xacro" / -->
-	<xacro:include filename="$(find jaco_model)/urdf/jaco_arm.xacro" />
+	<!--xacro:include filename="$(find jaco_model)/urdf/jaco_arm.xacro" /-->
+	<xacro:include filename="$(find kinova_description)/urdf/j2n6s300.xacro" />
 	<!-- Fix torso to base -->
-	<joint
-	  name="j_base_torso"
-      type="fixed">
-    <origin
-      xyz="-0.133 0.0 0.213"
-      rpy="0.0 0.0 0.0" />
-    <parent
-      link="base_link" />
-    <child
-      link="base_link_rb1_torso" />
-    <axis
-      xyz="0 0 0" />
-  </joint>
+	<!--joint name="j_base_torso" type="fixed">
+    <origin xyz="-0.133 0.0 0.213" rpy="0.0 0.0 0.0" />
+    <parent link="base_link" />
+    <child link="base_link_rb1_torso" />
+    <axis xyz="0 0 0" />
+  </joint-->
   <!-- temporary offset - until home seq can be changed -->
   <!-- 55 mm +X, 315 mm -Y, 100 mm +Z -->
-  <!-- Fix arm to torso -->
-  <joint
-	  name="j_torso_arm"
-      type="fixed">
-    <!-- origin
-      xyz="0.055 0.0 0.0755"
-      rpy="0.0 0.0 0.0" / -->
-    <origin
-      xyz="0.100 -0.315 0.1755"
-      rpy="0.0 0.0 0.0" />
-    <parent
-      link="link2_torso" />
-    <child
-      link="arm_link_base" />
-    <axis
-      xyz="0 0 0" />
+  <!-- Create link to fix arm to torso -->
+  <link name="link_torso_arm" />
+  <joint name="j_torso_arm" type="fixed">
+    <origin xyz="0.05 0.0 0.0" rpy="0.0 0.0 0.0" />
+    <parent link="torso_slider_link" />
+    <child link="link_torso_arm" />
+    <axis xyz="0 0 0" />
   </joint>
-  <link name="arm_link_base">
-  </link>
   <!-- Gazebo ros control pluggins -->
   <!-- xacro:ros_control/ -->
-  <!-- arm -->
-  <xacro:jaco_arm parent="arm_link_base"/>
+  <!-- Instance of Arm -->
+  <xacro:j2n6s300 base_parent="link_torso_arm" />
 </robot>

File: rb1_torso_description/robots/rb1_torso.urdf.xacro (robot description, xacro)
@@ -16,5 +16,5 @@
 	<xacro:property name="hq" value="false" />
 	<!-- RB-1 torso -->
-	<xacro:rb1_torso_3dof name="rb1_torso_3dof" hq="${hq}" />
+	<xacro:rb1_torso_3dof base_parent="rb1_base_link" hq="${hq}" />
 	<!-- Ixtion sensor in head -->
 	<!-- xacro:sensor_asus_xtion_pro name="xtion_head" parent="link2_head">
@@ -22,5 +22,5 @@
     </xacro:sensor_asus_xtion_pro -->
     <!-- RGBD sensor -->
-    <xacro:sensor_orbbec_astra name="head_camera" parent="head_tilt_link">
+    <xacro:sensor_orbbec_astra prefix="head_camera" parent="head_tilt_link" prefix_topic="head_rgbd_camera">
         <origin xyz="0.055 0.0125 0.028" rpy="0 0 0"/>
     </xacro:sensor_orbbec_astra>

File: rb1_torso_description/urdf/rb1_torso_3dof.urdf.xacro (robot description, xacro)
@@ -1,5 +1,4 @@
 <?xml version="1.0"?>
 <robot name="rb1_torso_3dof" xmlns:xacro="http://www.ros.org/wiki/xacro">
-  <!-- xacro:include filename="$(find rb1_torso_description)/urdf/rb1_torso_3dof.gazebo.xacro" / -->
   <xacro:property name="joint_effort_limit" value="100.0"/>
   <xacro:property name="joint_velocity_limit" value="3.0"/>
@@ -14,301 +13,270 @@
   <xacro:property name="head_tilt_joint_mechanical_reduction" value="320.0"/>
   <xacro:property name="head_tilt_joint_motor_torque_constant" value="1.0"/>
-  <xacro:macro name="rb1_torso_3dof" params="name hq">
-  <!-- Robot mechanical and motor parameters -->
-  <xacro:property name="PI" value="3.1415926535897931"/>
-  <!-- BASE_LINK -->
-  <link
-    name="torso_base_link">
-  </link>
-  <link name="torso_link">
-    <inertial>
-      <mass value="3.0" />
-      <origin xyz="0 0 0" />
-      <inertia  ixx="1.0" ixy="0.0"  ixz="0.0"  iyy="1.0"  iyz="0.0"  izz="1.0" />
-    </inertial>
-    <visual>
-       <origin xyz="0 0 0" rpy="0 0 0" />
-       <xacro:if value="${hq}">
-       <geometry>
-	     <mesh filename="package://rb1_torso_description/meshes/torsos/rb1v2_superior1.dae"/>
-       </geometry>
-       </xacro:if>
-       <xacro:unless value="${hq}">
-       <geometry>
-       <mesh filename="package://rb1_torso_description/meshes/torsos/rb1v2_superior1.stl"/>
-       </geometry>
-       </xacro:unless>
-       <material name="darkgrey">
-         <color rgba="0.1 0.1 0.1 1"/>
-       </material>
-    </visual>
-    <collision>
-       <origin xyz="0 0 0" rpy="0 0 0 " />
-       <geometry>
-         <mesh filename="package://rb1_torso_description/meshes/torsos/rb1v2_superior1.dae"/>
-       </geometry>
-    </collision>
-  </link>
-  <joint
-	  name="torso_joint"
-      type="fixed">
-    <origin
-      xyz="0.0 0.0 0.0"
-      rpy="0.0 0.0 0.0" />
-    <parent
-      link="torso_base_link" />
-    <child
-      link="torso_link" />
-    <axis
-      xyz="0 0 0" />
-  </joint>
-  <link name="torso_guide_link">
-    <inertial>
-      <mass value="2.0" />
-      <origin xyz="0 0 0" />
-      <inertia  ixx="1.0" ixy="0.0"  ixz="0.0"  iyy="1.0"  iyz="0.0"  izz="1.0" />
-    </inertial>
-    <visual>
-       <origin xyz="0 0 0" rpy="0 0 0" />
-       <xacro:if value="${hq}">
-       <geometry>
-	     <mesh filename="package://rb1_torso_description/meshes/torsos/rb1v2_guide.dae"/>
-       </geometry>
-       </xacro:if>
-       <xacro:unless value="${hq}">
-       <geometry>
-       <mesh filename="package://rb1_torso_description/meshes/torsos/rb1v2_guide.stl"/>
-       </geometry>
-       </xacro:unless>
-       <material name="darkgrey">
-         <color rgba="0.1 0.1 0.1 1"/>
-       </material>
-    </visual>
-    <collision>
-       <origin xyz="0 0 0" rpy="0 0 0 " />
-       <geometry>
-         <mesh filename="package://rb1_torso_description/meshes/torsos/rb1v2_guide.dae"/>
-       </geometry>
-    </collision>
-  </link>
-  <joint
-	  name="torso_guide_joint"
-      type="fixed">
-    <origin
-      xyz="0.0 0.0 0.0"
-      rpy="0.0 0.0 0.0" />
-    <parent
-      link="torso_link" />
-    <child
-      link="torso_guide_link" />
-    <axis
-      xyz="0 0 0" />
-  </joint>
-  <link name="torso_slider_link">
-    <inertial>
-      <mass value="2.0" />
-      <origin xyz="0 0 0" />
-      <inertia  ixx="1.0" ixy="0.0"  ixz="0.0"  iyy="1.0"  iyz="0.0"  izz="1.0" />
-    </inertial>
-    <visual>
-       <origin xyz="0 0 0" rpy="0 0 0" />
-       <xacro:if value="${hq}">
-       <geometry>
-	     <mesh filename="package://rb1_torso_description/meshes/torsos/rb1v2_superior2.dae"/>
-       </geometry>
-       </xacro:if>
-       <xacro:unless value="${hq}">
-       <geometry>
-       <mesh filename="package://rb1_torso_description/meshes/torsos/rb1v2_superior2.stl"/>
-       </geometry>
-       </xacro:unless>
-       <material name="darkgrey">
-         <color rgba="0.1 0.1 0.1 1"/>
-       </material>
-    </visual>
-    <collision>
-       <origin xyz="0 0 0" rpy="0 0 0 " />
-       <geometry>
-         <mesh filename="package://rb1_torso_description/meshes/torsos/rb1v2_superior2.dae"/>
-       </geometry>
-    </collision>
-  </link>
-  <joint
-	name="torso_slider_joint"
-	type="prismatic">
-	<!-- origin
-      xyz="0.078 0 0.016"
-      rpy="0.0 0.0 0.0" / -->
-	<origin
-      xyz="0.078 0 0.091"
-      rpy="0.0 0.0 0.0" />
-	<parent link="torso_link" />
-    <child link="torso_slider_link" />
-    <axis xyz="0 0 1" />
-    <limit effort="${joint_effort_limit_torso}" velocity="${joint_velocity_limit_torso}" upper="${0.360}" lower="${0}"/>
-    <dynamics damping="${joint_damping}" friction="${joint_friction}"/>
-  </joint>
-  <transmission name="torso_slider_trans">
-	 <type>transmission_interface/SimpleTransmission</type>
-     <joint name="torso_slider_joint">
-		 <hardwareInterface>EffortJointInterface</hardwareInterface>
-     </joint>
-     <actuator name="torso_slider_motor">
-        <mechanicalReduction>${torso_slider_joint_mechanical_reduction}</mechanicalReduction>
-		<motorTorqueConstant>${torso_slider_joint_motor_torque_constant}</motorTorqueConstant>
-	 </actuator>
-  </transmission>
-  <link name="torso_cover_link">
-    <inertial>
-      <mass value="1.0" />
-      <origin xyz="0 0 0" />
-      <inertia  ixx="1.0" ixy="0.0"  ixz="0.0"  iyy="1.0"  iyz="0.0"  izz="1.0" />
-    </inertial>
-    <visual>
-       <origin xyz="0 0 0" rpy="0 0 0" />
-       <xacro:if value="${hq}">
-       <geometry>
-	     <mesh filename="package://rb1_torso_description/meshes/torsos/rb1v2_rear_cover.dae"/>
-       </geometry>
-       </xacro:if>
-       <xacro:unless value="${hq}">
-       <geometry>
-       <mesh filename="package://rb1_torso_description/meshes/torsos/rb1v2_rear_cover.stl"/>
-       </geometry>
-       </xacro:unless>
-       <material name="darkgrey">
-         <color rgba="0.1 0.1 0.1 1"/>
-       </material>
-    </visual>
-    <collision>
-       <origin xyz="0 0 0" rpy="0 0 0 " />
-       <geometry>
-         <mesh filename="package://rb1_torso_description/meshes/torsos/rb1v2_rear_cover.dae"/>
-       </geometry>
-    </collision>
-  </link>
-  <joint
-	  name="torso_cover_joint"
-      type="fixed">
-    <!--origin
-      xyz="-0.164 0.0 0.064"
-      rpy="0.0 0.0 0.0" / -->
-    <origin
-      xyz="-0.164 0.0 0.0"
-      rpy="0.0 0.0 0.0" />
-    <parent
-      link="torso_slider_link" />
-    <child
-      link="torso_cover_link" />
-    <axis
-      xyz="0 0 0" />
-  </joint>
-  <link name="head_link">
-    <inertial>
-      <mass value="1.0" />
-      <origin xyz="0 0 0" />
-      <inertia  ixx="1.0" ixy="0.0"  ixz="0.0"  iyy="1.0"  iyz="0.0"  izz="1.0" />
-    </inertial>
-    <visual>
-       <origin xyz="0 0 0" rpy="0 0 0" />
-       <xacro:if value="${hq}">
-       <geometry>
-	     <mesh filename="package://rb1_torso_description/meshes/heads/rb1v2_head1.dae"/>
-       </geometry>
-       </xacro:if>
-       <xacro:unless value="${hq}">
-       <geometry>
-       <mesh filename="package://rb1_torso_description/meshes/heads/rb1v2_head1.stl"/>
-       </geometry>
-       </xacro:unless>
-       <material name="darkgrey">
-         <color rgba="0.1 0.1 0.1 1"/>
-       </material>
-    </visual>
-    <collision>
-       <origin xyz="0 0 0" rpy="0 0 0 " />
-       <geometry>
-         <mesh filename="package://rb1_torso_description/meshes/heads/rb1v2_head1.dae"/>
-       </geometry>
-    </collision>
-  </link>
-  <joint
-	name="head_pan_joint"
-	type="revolute">
-	<!-- origin
-      xyz="0.055 0.0 0.686"
-      rpy="0.0 0.0 0.0" / -->
-	<origin
-      xyz="0.055 0.0 0.621"
-      rpy="0.0 0.0 0.0" />
-	<parent link="torso_slider_link" />
-    <child link="head_link" />
-    <axis xyz="0 0 1" />
-    <limit effort="${joint_effort_limit}" velocity="${joint_velocity_limit}" upper="${PI/2}" lower="${-PI/2}"/>
-    <dynamics damping="${joint_damping}" friction="${joint_friction}"/>
-  </joint>
-  <transmission name="head_pan_trans">
-	 <type>transmission_interface/SimpleTransmission</type>
-     <joint name="head_pan_joint">
-        <hardwareInterface>EffortJointInterface</hardwareInterface>
-     </joint>
-     <actuator name="head_pan_motor">
-        <mechanicalReduction>${head_pan_joint_mechanical_reduction}</mechanicalReduction>
-		<motorTorqueConstant>${head_pan_joint_motor_torque_constant}</motorTorqueConstant>
-	 </actuator>
-  </transmission>
-  <link name="head_tilt_link">
-    <inertial>
-      <mass value="1.0" />
-      <origin xyz="0 0 0" />
-      <inertia  ixx="1.0" ixy="0.0"  ixz="0.0"  iyy="1.0"  iyz="0.0"  izz="1.0" />
-    </inertial>
-    <visual>
-       <origin xyz="0 0 0" rpy="0 0 0" />
-       <xacro:if value="${hq}">
-       <geometry>
-	     <mesh filename="package://rb1_torso_description/meshes/heads/rb1v2_head2.dae"/>
-       </geometry>
-       </xacro:if>
-       <xacro:unless value="${hq}">
-       <geometry>
-       <mesh filename="package://rb1_torso_description/meshes/heads/rb1v2_head2.stl"/>
-       </geometry>
-       </xacro:unless>
-       <material name="darkgrey">
-         <color rgba="0.1 0.1 0.1 1"/>
-       </material>
-    </visual>
-    <collision>
-       <origin xyz="0 0 0" rpy="0 0 0 " />
-       <geometry>
-         <mesh filename="package://rb1_torso_description/meshes/heads/rb1v2_head2.dae"/>
-       </geometry>
-    </collision>
-  </link>
-  <joint
-	name="head_tilt_joint"
-	type="revolute">
-	<origin
-      xyz="0.081 0.0 0.0"
-      rpy="0.0 0.0 0.0" />
-	<parent link="head_link" />
-    <child link="head_tilt_link" />
-    <!-- check -->
-    <!-- axis xyz="0 1 0" / -->
-    <axis xyz="0 -1 0"/>
-    <limit effort="${joint_effort_limit}" velocity="${joint_velocity_limit}" upper="${PI/4}" lower="${-PI/4}"/>
-    <dynamics damping="${joint_damping}" friction="${joint_friction}"/>
-  </joint>
-  <transmission name="head_tilt_trans">
-	 <type>transmission_interface/SimpleTransmission</type>
-     <joint name="head_tilt_joint">
-		<hardwareInterface>EffortJointInterface</hardwareInterface>
-	 </joint>
-     <actuator name="head_tilt_motor">
-        <mechanicalReduction>${head_tilt_joint_mechanical_reduction}</mechanicalReduction>
-		<motorTorqueConstant>${head_tilt_joint_motor_torque_constant}</motorTorqueConstant>
-	 </actuator>
-  </transmission>
+  <xacro:macro name="rb1_torso_3dof" params="base_parent hq">
+    <!-- Robot mechanical and motor parameters -->
+    <xacro:property name="PI" value="3.1415926535897931"/>
+    <!-- BASE_LINK -->
+    <link name="torso_base_link">
+    </link>
+    <!-- Fix torso to base -->
+    <joint name="j_base_torso" type="fixed">
+      <origin xyz="-0.133 0.0 0.213" rpy="0.0 0.0 0.0" />
+      <parent link="${base_parent}" />
+      <child link="torso_base_link" />
+      <axis xyz="0 0 0" />
+    </joint>
+    <link name="torso_link">
+      <inertial>
+        <mass value="3.0" />
+        <origin xyz="0 0 0" />
+        <inertia  ixx="1.0" ixy="0.0"  ixz="0.0"  iyy="1.0"  iyz="0.0"  izz="1.0" />
+      </inertial>
+      <visual>
+        <origin xyz="0 0 0" rpy="0 0 0" />
+        <xacro:if value="${hq}">
+        <geometry>
+        <mesh filename="package://rb1_torso_description/meshes/torsos/rb1v2_superior1.dae"/>
+        </geometry>
+        </xacro:if>
+        <xacro:unless value="${hq}">
+        <geometry>
+        <mesh filename="package://rb1_torso_description/meshes/torsos/rb1v2_superior1.stl"/>
+        </geometry>
+        </xacro:unless>
+        <material name="darkgrey">
+          <color rgba="0.1 0.1 0.1 1"/>
+        </material>
+      </visual>
+      <collision>
+        <origin xyz="0 0 0" rpy="0 0 0 " />
+        <geometry>
+          <mesh filename="package://rb1_torso_description/meshes/torsos/rb1v2_superior1.dae"/>
+        </geometry>
+      </collision>
+    </link>
+    <joint name="torso_joint" type="fixed">
+      <origin xyz="0.0 0.0 0.0" rpy="0.0 0.0 0.0" />
+      <parent link="torso_base_link" />
+      <child link="torso_link" />
+      <axis xyz="0 0 0" />
+    </joint>
+    <link name="torso_guide_link">
+      <inertial>
+        <mass value="2.0" />
+        <origin xyz="0 0 0" />
+        <inertia  ixx="1.0" ixy="0.0"  ixz="0.0"  iyy="1.0"  iyz="0.0"  izz="1.0" />
+      </inertial>
+      <visual>
+        <origin xyz="0 0 0" rpy="0 0 0" />
+        <xacro:if value="${hq}">
+        <geometry>
+        <mesh filename="package://rb1_torso_description/meshes/torsos/rb1v2_guide.dae"/>
+        </geometry>
+        </xacro:if>
+        <xacro:unless value="${hq}">
+        <geometry>
+        <mesh filename="package://rb1_torso_description/meshes/torsos/rb1v2_guide.stl"/>
+        </geometry>
+        </xacro:unless>
+        <material name="darkgrey">
+          <color rgba="0.1 0.1 0.1 1"/>
+        </material>
+      </visual>
+      <collision>
+        <origin xyz="0 0 0" rpy="0 0 0 " />
+        <geometry>
+          <mesh filename="package://rb1_torso_description/meshes/torsos/rb1v2_guide.dae"/>
+        </geometry>
+      </collision>
+    </link>
+    <joint
+      name="torso_guide_joint"
+        type="fixed">
+      <origin
+        xyz="0.0 0.0 0.0"
+        rpy="0.0 0.0 0.0" />
+      <parent
+        link="torso_link" />
+      <child
+        link="torso_guide_link" />
+      <axis
+        xyz="0 0 0" />
+    </joint>
+    <link name="torso_slider_link">
+      <inertial>
+        <mass value="2.0" />
+        <origin xyz="0 0 0" />
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