Commit message: New parameters to choose arm

File: rb1_description/robots/rb1_robot_j2n6s300.urdf (robot description, URDF)
Before this commit: robot rb1, 37 links, 36 joints
Links:
- removed link front_cover_link
- removed link mico_link_1
- removed link mico_link_2
- removed link mico_link_3
- removed link mico_link_4
- removed link mico_link_5
- removed link mico_link_base
- removed link mico_link_finger_1
- removed link mico_link_finger_2
- removed link mico_link_finger_3
- removed link mico_link_hand
- removed link orbbec_astra_cam_depth_frame
- removed link orbbec_astra_cam_depth_optical_frame
- removed link orbbec_astra_cam_link
- removed link orbbec_astra_cam_rgb_frame
- removed link orbbec_astra_cam_rgb_optical_frame
- added link arm_link_base
- added link jaco_api_origin
- added link jaco_end_effector
- added link jaco_link_1; collision box size=0.079 0.027 0.080; collision cylinder length=0.004 radius=0.02
- added link jaco_link_2; collision box size=0.411 0.082 0.027; collision cylinder length=0.056 radius=0.0395
- added link jaco_link_3; collision box size=0.13 0.084 0.02; collision box size=0.15 0.072 0.02
- added link jaco_link_4; collision cylinder length=0.030 radius=0.036; collision cylinder length=0.045 radius=0.032
- added link jaco_link_5; collision cylinder length=0.030 radius=0.036; collision cylinder length=0.045 radius=0.032
- added link jaco_link_base; collision box size=0.051 0.011 0.038; collision cylinder length=0.154 radius=0.042
- added link jaco_link_finger_1; collision box size=0.119 0.022 0.019; visual mesh filename=package://jaco_model/meshes/jaco_link_finger_1.dae
- added link jaco_link_finger_2; collision box size=0.119 0.022 0.019; visual mesh filename=package://jaco_model/meshes/jaco_link_finger_2.dae
- added link jaco_link_finger_3; collision box size=0.119 0.022 0.019; visual mesh filename=package://jaco_model/meshes/jaco_link_finger_3.dae
- added link jaco_link_hand; collision box size=0.01 0.03 0.07; collision cylinder length=0.02 radius=0.04
- link base_link: geometry collision mesh filename=package://rb1_base_description/meshes/bases/rb1_base_v0.dae; visual mesh filename=package://rb1_base_description/meshes/bases/rb1_base_v0.dae
- link hokuyo_laser_link: geometry collision box size=0.1 0.1 0.08; visual mesh filename=package://robotnik_sensors/meshes/hokuyo_urg_04lx.dae
Joints:
- removed joint front_cover_joint
- removed joint mico_joint_1
- removed joint mico_joint_2
- removed joint mico_joint_3
- removed joint mico_joint_4
- removed joint mico_joint_5
- removed joint mico_joint_6
- removed joint mico_joint_finger_1
- removed joint mico_joint_finger_2
- removed joint mico_joint_finger_3
- removed joint orbbec_astra_cam_depth_joint
- removed joint orbbec_astra_cam_depth_optical_joint
- removed joint orbbec_astra_cam_joint
- removed joint orbbec_astra_cam_rgb_joint
- removed joint orbbec_astra_cam_rgb_optical_joint
- added joint jaco_joint_1: type continuous, parent jaco_link_base, child jaco_link_1, origin xyz=0 0 0.1535 rpy=3.14159265359 0 3.14159265359, axis 0 0 -1, limit lower=-6.28318530718 upper=6.28318530718 effort=30 velocity=0.35
- added joint jaco_joint_2: type revolute, parent jaco_link_1, child jaco_link_2, origin xyz=0 0 -0.1185 rpy=-1.57079632679 3.14159265359 0, axis 0 0 1, limit lower=-3.14159265359 upper=0.0 effort=30 velocity=0.35
- added joint jaco_joint_3: type revolute, parent jaco_link_2, child jaco_link_3, origin xyz=0.41 0 0 rpy=3.14159265359 0 1.57079632679, axis 0 0 -1, limit lower=-3.92699081699 upper=0.785398163397 effort=30 velocity=0.35
- added joint jaco_joint_4: type continuous, parent jaco_link_3, child jaco_link_4, origin xyz=0.207 0 -0.01125 rpy=3.14159265359 1.57079632679 0, axis 0 0 -1, limit lower=-6.28318530718 upper=6.28318530718 effort=30 velocity=0.35
- added joint jaco_joint_5: type continuous, parent jaco_link_4, child jaco_link_5, origin xyz=0.0343 0 -0.06588 rpy=0 -0.959931088597 0, axis 0 0 -1, limit lower=-6.28318530718 upper=6.28318530718 effort=30 velocity=0.35
- added joint jaco_joint_6: type continuous, parent jaco_link_5, child jaco_link_hand, origin xyz=0.0343 0 -0.06588 rpy=-0.959931088597 0 1.57079632679, axis 0 0 -1, limit lower=-6.28318530718 upper=6.28318530718 effort=30 velocity=0.35
- added joint jaco_joint_base: type fixed, parent arm_link_base, child jaco_link_base, origin xyz=0 0 0 rpy=0 0 0, axis 0 0 0, limit lower=0 upper=0 effort=30 velocity=0.35
- added joint jaco_joint_finger_1: type revolute, parent jaco_link_hand, child jaco_link_finger_1, origin xyz=-0.03978 0 -0.10071 rpy=-1.7983 1.117 3.1416, axis 0 0 1, limit lower=0 upper=0.698131700798 effort=30 velocity=5
- added joint jaco_joint_finger_2: type revolute, parent jaco_link_hand, child jaco_link_finger_2, origin xyz=0.03569 -0.0216 -0.10071 rpy=-1.6222 1.117 -0.23615, axis 0 0 1, limit lower=0 upper=0.698131700798 effort=30 velocity=5
- added joint jaco_joint_finger_3: type revolute, parent jaco_link_hand, child jaco_link_finger_3, origin xyz=0.03569 0.0216 -0.10071 rpy=-1.5161 1.1459 0.23978, axis 0 0 1, limit lower=0 upper=0.698131700798 effort=30 velocity=5
- added joint jaco_link_base_to_api_origin: type fixed, parent jaco_link_base, child jaco_api_origin, origin xyz=0 0 0.028 rpy=0 0 0
- added joint jaco_link_hand_to_end_effector: type fixed, parent jaco_link_hand, child jaco_end_effector, origin xyz=0 0 -0.1687 rpy=0 3.14159265359 0
- joint hokuyo_laser_joint: origin xyz=0.223 0.0 0.159 rpy=0 3.1416 3.1416 -> xyz=0.220 0.0 0.170 rpy=0 3.1416 3.1416
- joint j11_rb1_torso: origin xyz=-0.164 0.0 0.0 rpy=0.0 0.0 0.0 -> xyz=-0.164 0.0 0.064 rpy=0.0 0.0 0.0
- joint j1_head: limit lower=-1.57079632679 upper=1.57079632679 effort=60.0 velocity=2.9217 -> lower=-1.57079632679 upper=1.57079632679 effort=100.0 velocity=3.0; origin xyz=0.055 0.0 0.621 rpy=0.0 0.0 0.0 -> xyz=0.055 0.0 0.686 rpy=0.0 0.0 0.0
- joint j1_torso: origin xyz=0.078 0 0.091 rpy=0.0 0.0 0.0 -> xyz=0.078 0 0.016 rpy=0.0 0.0 0.0
- joint j2_head: limit lower=-0.785398163397 upper=0.785398163397 effort=60.0 velocity=2.9217 -> lower=-0.785398163397 upper=0.785398163397 effort=100.0 velocity=3.0
- joint j_torso_arm: child mico_link_base -> arm_link_base; origin xyz=0.055 0.0 0.010 rpy=0.0 0.0 0.0 -> xyz=0.100 -0.315 0.1755 rpy=0.0 0.0 0.0
- joint joint_left_wheel: origin xyz=0.0 0.217 0.051 rpy=0 0 0 -> xyz=0.0 0.183 0.051 rpy=0 0 0
- joint joint_omni_back_wheel: origin xyz=-0.195 0.0 0.0265 rpy=0 0 0 -> xyz=-0.185 0.0 0.0265 rpy=0 0 0
- joint joint_omni_front_left_wheel: origin xyz=0.133 0.148 0.0265 rpy=0 0 0 -> xyz=0.133 0.142 0.0265 rpy=0 0 0
- joint joint_omni_front_right_wheel: origin xyz=0.133 -0.148 0.0265 rpy=0 0 0 -> xyz=0.133 -0.142 0.0265 rpy=0 0 0
- joint joint_right_wheel: origin xyz=0.0 -0.217 0.051 rpy=0 0 0 -> xyz=0.0 -0.183 0.051 rpy=0 0 0

File: rb1_torso_description/urdf/rb1_torso_3dof.gazebo.xacro (robot description, xacro)
@@ -1,4 +1,4 @@
 <?xml version="1.0"?>
-<robot xmlns:xacro="http://ros.org/wiki/xacro">
+<robot xmlns:xacro="http://www.ros.org/wiki/xacro">
   <!-- ros control plugin -->
   <xacro:macro name="ros_control">
