Commit message: Add j2s7s200 support

File: rb1_description/robots/rb1_robot_j2s7s200.urdf.xacro (robot description, xacro)
@@ -49,5 +49,5 @@
 	<!-- Fix arm to torso -->
 	<joint name="j_torso_arm" type="fixed">
-		<origin xyz="0.05 0.0 0.0" rpy="0.0 0.0 0.0" />
+		<origin xyz="0.05 0.0 0.0" rpy="0.0 0.0 ${PI/2}" />
 		<parent link="torso_slider_link" />
 		<child link="arm_base_link" />

Commit message: Lot of fixes
Correction on namespaces
Correction on controllers
Correction on URDF arm position

File: rb1_description/robots/rb1_robot_j2s7s200.urdf.xacro (robot description, xacro)
@@ -49,5 +49,5 @@
 	<!-- Fix arm to torso -->
 	<joint name="j_torso_arm" type="fixed">
-		<origin xyz="0.05 0.0 0.0" rpy="0.0 0.0 ${PI/2}" />
+		<origin xyz="0.05 0.0 0.0" rpy="0.0 0.0 0.0" />
 		<parent link="torso_slider_link" />
 		<child link="arm_base_link" />

Commit message: Add camera frame link

File: rb1_description/robots/rb1_robot_j2s7s200.urdf.xacro (robot description, xacro)
@@ -54,3 +54,19 @@
 		<axis xyz="0 0 0" />
 	</joint>
+	<!-- Front camera scan link -->
+	<link name="$(arg prefix)front_rgbd_camera_depth_optical_scan_frame" />
+	<joint name="$(arg prefix)front_rgbd_camera_depth_optical_scan_joint" type="fixed">
+		<origin xyz="0 0 0" rpy="${PI/2} 0 0" />
+		<parent link="$(arg prefix)front_rgbd_camera_depth_optical_frame" />
+		<child link="$(arg prefix)front_rgbd_camera_depth_optical_scan_frame" />
+		<axis xyz="0 0 0" />
+	</joint>
+	<!-- Torso camera scan link -->
+	<link name="$(arg prefix)torso_rgbd_camera_depth_optical_scan_frame" />
+	<joint name="$(arg prefix)torso_rgbd_camera_depth_optical_scan_joint" type="fixed">
+		<origin xyz="0 0 0" rpy="${PI/2} 0 0" />
+		<parent link="$(arg prefix)torso_rgbd_camera_depth_optical_frame" />
+		<child link="$(arg prefix)torso_rgbd_camera_depth_optical_scan_frame" />
+		<axis xyz="0 0 0" />
+	</joint>
 </robot>

Commit message: Remove redundant links

File: rb1_description/robots/rb1_robot_j2s7s200.urdf.xacro (robot description, xacro)
@@ -54,19 +54,3 @@
 		<axis xyz="0 0 0" />
 	</joint>
-	<!-- Front camera scan link -->
-	<link name="$(arg prefix)front_rgbd_camera_depth_optical_scan_frame" />
-	<joint name="$(arg prefix)front_rgbd_camera_depth_optical_scan_joint" type="fixed">
-		<origin xyz="0 0 0" rpy="${PI/2} 0 0" />
-		<parent link="$(arg prefix)front_rgbd_camera_depth_optical_frame" />
-		<child link="$(arg prefix)front_rgbd_camera_depth_optical_scan_frame" />
-		<axis xyz="0 0 0" />
-	</joint>
-	<!-- Torso camera scan link -->
-	<link name="$(arg prefix)torso_rgbd_camera_depth_optical_scan_frame" />
-	<joint name="$(arg prefix)torso_rgbd_camera_depth_optical_scan_joint" type="fixed">
-		<origin xyz="0 0 0" rpy="${PI/2} 0 0" />
-		<parent link="$(arg prefix)torso_rgbd_camera_depth_optical_frame" />
-		<child link="$(arg prefix)torso_rgbd_camera_depth_optical_scan_frame" />
-		<axis xyz="0 0 0" />
-	</joint>
 </robot>
