Commit message: urdf and meshes of the new torso. xtion x orbbec

File: rb1_torso_description/robots/rb1_torso_standalone_v0.urdf.xacro (robot description, xacro)
@@ -19,10 +19,7 @@
 	<xacro:rb1_torso_3dof name="rb1_torso_3dof" hq="${hq}" />
 	<!-- Ixtion sensor in head -->
-	<!-- xacro:sensor_asus_xtion_pro name="xtion_head" parent="link2_head">
+	<xacro:sensor_asus_xtion_pro name="xtion_head" parent="link2_head">
         <origin xyz="0.055 0.000 0.028" rpy="0 0 0"/>
-    </xacro:sensor_asus_xtion_pro -->
-    <xacro:sensor_orbbec_astra name="orbbec_astra" parent="link2_head">
-        <origin xyz="0.055 0.0125 0.028" rpy="0 0 0"/>
-    </xacro:sensor_orbbec_astra>
+   </xacro:sensor_asus_xtion_pro>
 	<!-- Gazebo ros control plugins -->
 	<!-- xacro:ros_control/ -->

File: rb1_torso_description/robots/rb1_torso_v0.urdf.xacro (robot description, xacro)
@@ -7,5 +7,4 @@
 	<!-- Import RB1 arm elements -->
 	<xacro:include filename="$(find rb1_torso_description)/urdf/rb1_torso_3dof.urdf.xacro" />
-	<xacro:include filename="$(find rb1_torso_description)/urdf/rb1_torso_3dof.gazebo.xacro" />
 	<!-- Import all available sensors -->
 	<xacro:include filename="$(find robotnik_sensors)/urdf/all_sensors.urdf.xacro" />
@@ -19,10 +18,7 @@
 	<xacro:rb1_torso_3dof name="rb1_torso_3dof" hq="${hq}" />
 	<!-- Ixtion sensor in head -->
-	<!-- xacro:sensor_asus_xtion_pro name="xtion_head" parent="link2_head">
+	<xacro:sensor_asus_xtion_pro name="xtion_head" parent="link2_head">
         <origin xyz="0.055 0.000 0.028" rpy="0 0 0"/>
-    </xacro:sensor_asus_xtion_pro -->
-    <xacro:sensor_orbbec_astra name="orbbec_astra" parent="link2_head">
-        <origin xyz="0.055 0.0125 0.028" rpy="0 0 0"/>
-    </xacro:sensor_orbbec_astra>
+   </xacro:sensor_asus_xtion_pro>
 	<!-- Gazebo ros control plugins -->
 	<!-- xacro:ros_control/ -->

File: rb1_torso_description/urdf/rb1_torso_3dof_v0.urdf.xacro (robot description, xacro)
@@ -31,20 +31,20 @@
        <xacro:if value="${hq}">
        <geometry>
-	     <mesh filename="package://rb1_torso_description/meshes/torsos/rb1v2_superior1.dae"/>
-       </geometry>
-       </xacro:if>
-       <xacro:unless value="${hq}">
-       <geometry>
-       <mesh filename="package://rb1_torso_description/meshes/torsos/rb1v2_superior1.stl"/>
-       </geometry>
-       </xacro:unless>
-       <material name="darkgrey">
-         <color rgba="0.1 0.1 0.1 1"/>
-       </material>
-    </visual>
-    <collision>
-       <origin xyz="0 0 0" rpy="0 0 0 " />
-       <geometry>
-         <mesh filename="package://rb1_torso_description/meshes/torsos/rb1v2_superior1.dae"/>
+	     <mesh filename="package://rb1_torso_description/meshes/torsos/rb1_lower.dae"/>
+       </geometry>
+       </xacro:if>
+       <xacro:unless value="${hq}">
+       <geometry>
+       <mesh filename="package://rb1_torso_description/meshes/torsos/rb1_lower.stl"/>
+       </geometry>
+       </xacro:unless>
+       <material name="darkgrey">
+         <color rgba="0.1 0.1 0.1 1"/>
+       </material>
+    </visual>
+    <collision>
+       <origin xyz="0 0 0" rpy="0 0 0 " />
+       <geometry>
+         <mesh filename="package://rb1_torso_description/meshes/torsos/rb1_lower.dae"/>
        </geometry>
     </collision>
@@ -63,5 +63,5 @@
       xyz="0 0 0" />
   </joint>
-  <link name="link1_guide">
+  <link name="link2_torso">
     <inertial>
       <mass value="2.0" />
@@ -73,62 +73,20 @@
        <xacro:if value="${hq}">
        <geometry>
-	     <mesh filename="package://rb1_torso_description/meshes/torsos/rb1v2_guide.dae"/>
-       </geometry>
-       </xacro:if>
-       <xacro:unless value="${hq}">
-       <geometry>
-       <mesh filename="package://rb1_torso_description/meshes/torsos/rb1v2_guide.stl"/>
-       </geometry>
-       </xacro:unless>
-       <material name="darkgrey">
-         <color rgba="0.1 0.1 0.1 1"/>
-       </material>
-    </visual>
-    <collision>
-       <origin xyz="0 0 0" rpy="0 0 0 " />
-       <geometry>
-         <mesh filename="package://rb1_torso_description/meshes/torsos/rb1v2_guide.dae"/>
-       </geometry>
-    </collision>
-  </link>
-  <joint
-	  name="j00_rb1_torso"
-      type="fixed">
-    <origin
-      xyz="0.0 0.0 0.0"
-      rpy="0.0 0.0 0.0" />
-    <parent
-      link="link1_torso" />
-    <child
-      link="link1_guide" />
-    <axis
-      xyz="0 0 0" />
-  </joint>
-  <link name="link2_torso">
-    <inertial>
-      <mass value="2.0" />
-      <origin xyz="0 0 0" />
-      <inertia  ixx="1.0" ixy="0.0"  ixz="0.0"  iyy="1.0"  iyz="0.0"  izz="1.0" />
-    </inertial>
-    <visual>
-       <origin xyz="0 0 0" rpy="0 0 0" />
-       <xacro:if value="${hq}">
-       <geometry>
-	     <mesh filename="package://rb1_torso_description/meshes/torsos/rb1v2_superior2.dae"/>
-       </geometry>
-       </xacro:if>
-       <xacro:unless value="${hq}">
-       <geometry>
-       <mesh filename="package://rb1_torso_description/meshes/torsos/rb1v2_superior2.stl"/>
-       </geometry>
-       </xacro:unless>
-       <material name="darkgrey">
-         <color rgba="0.1 0.1 0.1 1"/>
-       </material>
-    </visual>
-    <collision>
-       <origin xyz="0 0 0" rpy="0 0 0 " />
-       <geometry>
-         <mesh filename="package://rb1_torso_description/meshes/torsos/rb1v2_superior2.dae"/>
+	     <mesh filename="package://rb1_torso_description/meshes/torsos/rb1_upper.dae"/>
+       </geometry>
+       </xacro:if>
+       <xacro:unless value="${hq}">
+       <geometry>
+       <mesh filename="package://rb1_torso_description/meshes/torsos/rb1_upper.stl"/>
+       </geometry>
+       </xacro:unless>
+       <material name="darkgrey">
+         <color rgba="0.1 0.1 0.1 1"/>
+       </material>
+    </visual>
+    <collision>
+       <origin xyz="0 0 0" rpy="0 0 0 " />
+       <geometry>
+         <mesh filename="package://rb1_torso_description/meshes/torsos/rb1_upper.dae"/>
        </geometry>
     </collision>
@@ -138,5 +96,5 @@
 	type="prismatic">
 	<origin
-      xyz="0.078 0 0.016"
+      xyz="0 0 0"
       rpy="0.0 0.0 0.0" />
 	<parent link="link1_torso" />
@@ -156,5 +114,5 @@
 	 </actuator>
   </transmission>
-  <link name="link2_cover">
+  <link name="link1_head">
     <inertial>
       <mass value="1.0" />
@@ -166,62 +124,20 @@
        <xacro:if value="${hq}">
        <geometry>
-	     <mesh filename="package://rb1_torso_description/meshes/torsos/rb1v2_rear_cover.dae"/>
-       </geometry>
-       </xacro:if>
-       <xacro:unless value="${hq}">
-       <geometry>
-       <mesh filename="package://rb1_torso_description/meshes/torsos/rb1v2_rear_cover.stl"/>
-       </geometry>
-       </xacro:unless>
-       <material name="darkgrey">
-         <color rgba="0.1 0.1 0.1 1"/>
-       </material>
-    </visual>
-    <collision>
-       <origin xyz="0 0 0" rpy="0 0 0 " />
-       <geometry>
-         <mesh filename="package://rb1_torso_description/meshes/torsos/rb1v2_rear_cover.dae"/>
-       </geometry>
-    </collision>
-  </link>
-  <joint
-	  name="j11_rb1_torso"
-      type="fixed">
-    <origin
-      xyz="-0.164 0.0 0.064"
-      rpy="0.0 0.0 0.0" />
-    <parent
-      link="link2_torso" />
-    <child
-      link="link2_cover" />
-    <axis
-      xyz="0 0 0" />
-  </joint>
-  <link name="link1_head">
-    <inertial>
-      <mass value="1.0" />
-      <origin xyz="0 0 0" />
-      <inertia  ixx="1.0" ixy="0.0"  ixz="0.0"  iyy="1.0"  iyz="0.0"  izz="1.0" />
-    </inertial>
-    <visual>
-       <origin xyz="0 0 0" rpy="0 0 0" />
-       <xacro:if value="${hq}">
-       <geometry>
-	     <mesh filename="package://rb1_torso_description/meshes/heads/rb1v2_head1.dae"/>
-       </geometry>
-       </xacro:if>
-       <xacro:unless value="${hq}">
-       <geometry>
-       <mesh filename="package://rb1_torso_description/meshes/heads/rb1v2_head1.stl"/>
-       </geometry>
-       </xacro:unless>
-       <material name="darkgrey">
-         <color rgba="0.1 0.1 0.1 1"/>
-       </material>
-    </visual>
-    <collision>
-       <origin xyz="0 0 0" rpy="0 0 0 " />
-       <geometry>
-         <mesh filename="package://rb1_torso_description/meshes/heads/rb1v2_head1.dae"/>
+	     <mesh filename="package://rb1_torso_description/meshes/heads/head1.dae"/>
+       </geometry>
+       </xacro:if>
+       <xacro:unless value="${hq}">
+       <geometry>
+       <mesh filename="package://rb1_torso_description/meshes/heads/head1.stl"/>
+       </geometry>
+       </xacro:unless>
+       <material name="darkgrey">
+         <color rgba="0.1 0.1 0.1 1"/>
+       </material>
+    </visual>
+    <collision>
+       <origin xyz="0 0 0" rpy="0 0 0 " />
+       <geometry>
+         <mesh filename="package://rb1_torso_description/meshes/heads/head1.dae"/>
        </geometry>
     </collision>
@@ -231,5 +147,5 @@
 	type="revolute">
 	<origin
-      xyz="0.055 0.0 0.686"
+      xyz="0.010 0.0 0.940"
       rpy="0.0 0.0 0.0" />
 	<parent link="link2_torso" />
@@ -259,20 +175,20 @@
        <xacro:if value="${hq}">
        <geometry>
-	     <mesh filename="package://rb1_torso_description/meshes/heads/rb1v2_head2.dae"/>
-       </geometry>
-       </xacro:if>
-       <xacro:unless value="${hq}">
-       <geometry>
-       <mesh filename="package://rb1_torso_description/meshes/heads/rb1v2_head2.stl"/>
-       </geometry>
-       </xacro:unless>
-       <material name="darkgrey">
-         <color rgba="0.1 0.1 0.1 1"/>
-       </material>
-    </visual>
-    <collision>
-       <origin xyz="0 0 0" rpy="0 0 0 " />
-       <geometry>
-         <mesh filename="package://rb1_torso_description/meshes/heads/rb1v2_head2.dae"/>
+	     <mesh filename="package://rb1_torso_description/meshes/heads/head2.dae"/>
+       </geometry>
+       </xacro:if>
+       <xacro:unless value="${hq}">
+       <geometry>
+       <mesh filename="package://rb1_torso_description/meshes/heads/head2.stl"/>
+       </geometry>
+       </xacro:unless>
+       <material name="darkgrey">
+         <color rgba="0.1 0.1 0.1 1"/>
+       </material>
+    </visual>
+    <collision>
+       <origin xyz="0 0 0" rpy="0 0 0 " />
+       <geometry>
+         <mesh filename="package://rb1_torso_description/meshes/heads/head2.dae"/>
        </geometry>
     </collision>
@@ -282,5 +198,5 @@
 	type="revolute">
 	<origin
-      xyz="0.081 0.0 0.0"
+      xyz="0.105 0.0 0.0"
       rpy="0.0 0.0 0.0" />
 	<parent link="link1_head" />
