Commit message: updated meshes and xacro to latest rb1 version

File: rb1_torso_description/robots/rb1_torso.urdf.xacro (robot description, xacro)
@@ -14,5 +14,5 @@
 	<xacro:property name="PI" value="3.1415926535897931"/>
 	<!-- Flag to select the high or low quality model -->
-	<xacro:property name="hq" value="true" />
+	<xacro:property name="hq" value="false" />
 	<!-- RB-1 torso -->
 	<xacro:rb1_torso_3dof name="rb1_torso_3dof" hq="${hq}" />

File: rb1_torso_description/urdf/rb1_torso_3dof.urdf.xacro (robot description, xacro)
@@ -137,6 +137,9 @@
 	name="j1_torso"
 	type="prismatic">
+	<!-- origin
+      xyz="0.078 0 0.016"
+      rpy="0.0 0.0 0.0" / -->
 	<origin
-      xyz="0.078 0 0.016"
+      xyz="0.078 0 0.091"
       rpy="0.0 0.0 0.0" />
 	<parent link="link1_torso" />
@@ -188,6 +191,9 @@
 	  name="j11_rb1_torso"
       type="fixed">
+    <!--origin
+      xyz="-0.164 0.0 0.064"
+      rpy="0.0 0.0 0.0" / -->
     <origin
-      xyz="-0.164 0.0 0.064"
+      xyz="-0.164 0.0 0.0"
       rpy="0.0 0.0 0.0" />
     <parent
@@ -230,6 +236,9 @@
 	name="j1_head"
 	type="revolute">
+	<!-- origin
+      xyz="0.055 0.0 0.686"
+      rpy="0.0 0.0 0.0" / -->
 	<origin
-      xyz="0.055 0.0 0.686"
+      xyz="0.055 0.0 0.621"
       rpy="0.0 0.0 0.0" />
 	<parent link="link2_torso" />

Commit message: rb1_torso_description: changed joint and links names to something more readable

File: rb1_torso_description/robots/rb1_torso.urdf.xacro (robot description, xacro)
@@ -22,5 +22,5 @@
     </xacro:sensor_asus_xtion_pro -->
     <!-- RGBD sensor -->
-    <xacro:sensor_orbbec_astra name="head_camera" parent="link2_head">
+    <xacro:sensor_orbbec_astra name="head_camera" parent="torso_head_tilt_link">
         <origin xyz="0.055 0.0125 0.028" rpy="0 0 0"/>
     </xacro:sensor_orbbec_astra>

File: rb1_torso_description/urdf/rb1_torso_3dof.urdf.xacro (robot description, xacro)
@@ -8,10 +8,10 @@
   <xacro:property name="joint_damping" value="0.5"/>
   <xacro:property name="joint_friction" value="0.5"/>
-  <xacro:property name="j1_torso_mechanical_reduction" value="320.0"/>
-  <xacro:property name="j1_torso_motor_torque_constant" value="1.0"/>
-  <xacro:property name="j1_head_mechanical_reduction" value="320.0"/>
-  <xacro:property name="j1_head_motor_torque_constant" value="1.0"/>
-  <xacro:property name="j2_head_mechanical_reduction" value="320.0"/>
-  <xacro:property name="j2_head_motor_torque_constant" value="1.0"/>
+  <xacro:property name="torso_slider_joint_mechanical_reduction" value="320.0"/>
+  <xacro:property name="torso_slider_joint_motor_torque_constant" value="1.0"/>
+  <xacro:property name="torso_head_pan_joint_mechanical_reduction" value="320.0"/>
+  <xacro:property name="torso_head_pan_joint_motor_torque_constant" value="1.0"/>
+  <xacro:property name="torso_head_tilt_joint_mechanical_reduction" value="320.0"/>
+  <xacro:property name="torso_head_tilt_joint_motor_torque_constant" value="1.0"/>
   <xacro:macro name="rb1_torso_3dof" params="name hq">
   <!-- Robot mechanical and motor parameters -->
@@ -19,7 +19,7 @@
   <!-- BASE_LINK -->
   <link
-    name="base_link_rb1_torso">
-  </link>
-  <link name="link1_torso">
+    name="torso_base_link">
+  </link>
+  <link name="torso_link">
     <inertial>
       <mass value="3.0" />
@@ -51,5 +51,5 @@
   </link>
   <joint
-	  name="j0_rb1_torso"
+	  name="torso_joint"
       type="fixed">
     <origin
@@ -57,11 +57,11 @@
       rpy="0.0 0.0 0.0" />
     <parent
-      link="base_link_rb1_torso" />
+      link="torso_base_link" />
     <child
-      link="link1_torso" />
+      link="torso_link" />
     <axis
       xyz="0 0 0" />
   </joint>
-  <link name="link1_guide">
+  <link name="torso_guide_link">
     <inertial>
       <mass value="2.0" />
@@ -93,5 +93,5 @@
   </link>
   <joint
-	  name="j00_rb1_torso"
+	  name="torso_guide_joint"
       type="fixed">
     <origin
@@ -99,11 +99,11 @@
       rpy="0.0 0.0 0.0" />
     <parent
-      link="link1_torso" />
+      link="torso_link" />
     <child
-      link="link1_guide" />
+      link="torso_guide_link" />
     <axis
       xyz="0 0 0" />
   </joint>
-  <link name="link2_torso">
+  <link name="torso_slider_link">
     <inertial>
       <mass value="2.0" />
@@ -135,5 +135,5 @@
   </link>
   <joint
-	name="j1_torso"
+	name="torso_slider_joint"
 	type="prismatic">
 	<!-- origin
@@ -143,21 +143,21 @@
       xyz="0.078 0 0.091"
       rpy="0.0 0.0 0.0" />
-	<parent link="link1_torso" />
-    <child link="link2_torso" />
+	<parent link="torso_link" />
+    <child link="torso_slider_link" />
     <axis xyz="0 0 1" />
     <limit effort="${joint_effort_limit_torso}" velocity="${joint_velocity_limit_torso}" upper="${0.360}" lower="${0}"/>
     <dynamics damping="${joint_damping}" friction="${joint_friction}"/>
   </joint>
-  <transmission name="j1_torso_trans">
+  <transmission name="torso_slider_trans">
 	 <type>transmission_interface/SimpleTransmission</type>
-     <joint name="j1_torso">
+     <joint name="torso_slider_joint">
 		 <hardwareInterface>EffortJointInterface</hardwareInterface>
      </joint>
-     <actuator name="j1_torso_motor">
-        <mechanicalReduction>${j1_torso_mechanical_reduction}</mechanicalReduction>
-		<motorTorqueConstant>${j1_torso_motor_torque_constant}</motorTorqueConstant>
+     <actuator name="torso_slider_motor">
+        <mechanicalReduction>${torso_slider_joint_mechanical_reduction}</mechanicalReduction>
+		<motorTorqueConstant>${torso_slider_joint_motor_torque_constant}</motorTorqueConstant>
 	 </actuator>
   </transmission>
-  <link name="link2_cover">
+  <link name="torso_cover_link">
     <inertial>
       <mass value="1.0" />
@@ -189,5 +189,5 @@
   </link>
   <joint
-	  name="j11_rb1_torso"
+	  name="torso_cover_joint"
       type="fixed">
     <!--origin
@@ -198,11 +198,11 @@
       rpy="0.0 0.0 0.0" />
     <parent
-      link="link2_torso" />
+      link="torso_slider_link" />
     <child
-      link="link2_cover" />
+      link="torso_cover_link" />
     <axis
       xyz="0 0 0" />
   </joint>
-  <link name="link1_head">
+  <link name="torso_head_link">
     <inertial>
       <mass value="1.0" />
@@ -234,5 +234,5 @@
   </link>
   <joint
-	name="j1_head"
+	name="torso_head_pan_joint"
 	type="revolute">
 	<!-- origin
@@ -242,21 +242,21 @@
       xyz="0.055 0.0 0.621"
       rpy="0.0 0.0 0.0" />
-	<parent link="link2_torso" />
-    <child link="link1_head" />
+	<parent link="torso_slider_link" />
+    <child link="torso_head_link" />
     <axis xyz="0 0 1" />
     <limit effort="${joint_effort_limit}" velocity="${joint_velocity_limit}" upper="${PI/2}" lower="${-PI/2}"/>
     <dynamics damping="${joint_damping}" friction="${joint_friction}"/>
   </joint>
-  <transmission name="j1_head_trans">
+  <transmission name="torso_head_pan_trans">
 	 <type>transmission_interface/SimpleTransmission</type>
-     <joint name="j1_head">
+     <joint name="torso_head_pan_joint">
         <hardwareInterface>EffortJointInterface</hardwareInterface>
      </joint>
-     <actuator name="j1_head_motor">
-        <mechanicalReduction>${j1_head_mechanical_reduction}</mechanicalReduction>
-		<motorTorqueConstant>${j1_head_motor_torque_constant}</motorTorqueConstant>
+     <actuator name="torso_head_pan_motor">
+        <mechanicalReduction>${torso_head_pan_joint_mechanical_reduction}</mechanicalReduction>
+		<motorTorqueConstant>${torso_head_pan_joint_motor_torque_constant}</motorTorqueConstant>
 	 </actuator>
   </transmission>
-  <link name="link2_head">
+  <link name="torso_head_tilt_link">
     <inertial>
       <mass value="1.0" />
@@ -288,11 +288,11 @@
   </link>
   <joint
-	name="j2_head"
+	name="torso_head_tilt_joint"
 	type="revolute">
 	<origin
       xyz="0.081 0.0 0.0"
       rpy="0.0 0.0 0.0" />
-	<parent link="link1_head" />
-    <child link="link2_head" />
+	<parent link="torso_head_link" />
+    <child link="torso_head_tilt_link" />
     <!-- check -->
     <!-- axis xyz="0 1 0" / -->
@@ -301,12 +301,12 @@
     <dynamics damping="${joint_damping}" friction="${joint_friction}"/>
   </joint>
-  <transmission name="j2_head_trans">
+  <transmission name="torso_head_tilt_trans">
 	 <type>transmission_interface/SimpleTransmission</type>
-     <joint name="j2_head">
+     <joint name="torso_head_tilt_joint">
 		<hardwareInterface>EffortJointInterface</hardwareInterface>
 	 </joint>
-     <actuator name="j2_head_motor">
-        <mechanicalReduction>${j2_head_mechanical_reduction}</mechanicalReduction>
-		<motorTorqueConstant>${j2_head_motor_torque_constant}</motorTorqueConstant>
+     <actuator name="torso_head_tilt_motor">
+        <mechanicalReduction>${torso_head_tilt_joint_mechanical_reduction}</mechanicalReduction>
+		<motorTorqueConstant>${torso_head_tilt_joint_motor_torque_constant}</motorTorqueConstant>
 	 </actuator>
   </transmission>

Commit message: rb1_torso: renamed torso_head to head

File: rb1_torso_description/robots/rb1_torso.urdf.xacro (robot description, xacro)
@@ -22,5 +22,5 @@
     </xacro:sensor_asus_xtion_pro -->
     <!-- RGBD sensor -->
-    <xacro:sensor_orbbec_astra name="head_camera" parent="torso_head_tilt_link">
+    <xacro:sensor_orbbec_astra name="head_camera" parent="head_tilt_link">
         <origin xyz="0.055 0.0125 0.028" rpy="0 0 0"/>
     </xacro:sensor_orbbec_astra>

File: rb1_torso_description/urdf/rb1_torso_3dof.urdf.xacro (robot description, xacro)
@@ -10,8 +10,8 @@
   <xacro:property name="torso_slider_joint_mechanical_reduction" value="320.0"/>
   <xacro:property name="torso_slider_joint_motor_torque_constant" value="1.0"/>
-  <xacro:property name="torso_head_pan_joint_mechanical_reduction" value="320.0"/>
-  <xacro:property name="torso_head_pan_joint_motor_torque_constant" value="1.0"/>
-  <xacro:property name="torso_head_tilt_joint_mechanical_reduction" value="320.0"/>
-  <xacro:property name="torso_head_tilt_joint_motor_torque_constant" value="1.0"/>
+  <xacro:property name="head_pan_joint_mechanical_reduction" value="320.0"/>
+  <xacro:property name="head_pan_joint_motor_torque_constant" value="1.0"/>
+  <xacro:property name="head_tilt_joint_mechanical_reduction" value="320.0"/>
+  <xacro:property name="head_tilt_joint_motor_torque_constant" value="1.0"/>
   <xacro:macro name="rb1_torso_3dof" params="name hq">
   <!-- Robot mechanical and motor parameters -->
@@ -204,5 +204,5 @@
       xyz="0 0 0" />
   </joint>
-  <link name="torso_head_link">
+  <link name="head_link">
     <inertial>
       <mass value="1.0" />
@@ -234,5 +234,5 @@
   </link>
   <joint
-	name="torso_head_pan_joint"
+	name="head_pan_joint"
 	type="revolute">
 	<!-- origin
@@ -243,20 +243,20 @@
       rpy="0.0 0.0 0.0" />
 	<parent link="torso_slider_link" />
-    <child link="torso_head_link" />
+    <child link="head_link" />
     <axis xyz="0 0 1" />
     <limit effort="${joint_effort_limit}" velocity="${joint_velocity_limit}" upper="${PI/2}" lower="${-PI/2}"/>
     <dynamics damping="${joint_damping}" friction="${joint_friction}"/>
   </joint>
-  <transmission name="torso_head_pan_trans">
+  <transmission name="head_pan_trans">
 	 <type>transmission_interface/SimpleTransmission</type>
-     <joint name="torso_head_pan_joint">
+     <joint name="head_pan_joint">
         <hardwareInterface>EffortJointInterface</hardwareInterface>
      </joint>
-     <actuator name="torso_head_pan_motor">
-        <mechanicalReduction>${torso_head_pan_joint_mechanical_reduction}</mechanicalReduction>
-		<motorTorqueConstant>${torso_head_pan_joint_motor_torque_constant}</motorTorqueConstant>
+     <actuator name="head_pan_motor">
+        <mechanicalReduction>${head_pan_joint_mechanical_reduction}</mechanicalReduction>
+		<motorTorqueConstant>${head_pan_joint_motor_torque_constant}</motorTorqueConstant>
 	 </actuator>
   </transmission>
-  <link name="torso_head_tilt_link">
+  <link name="head_tilt_link">
     <inertial>
       <mass value="1.0" />
@@ -288,11 +288,11 @@
   </link>
   <joint
-	name="torso_head_tilt_joint"
+	name="head_tilt_joint"
 	type="revolute">
 	<origin
       xyz="0.081 0.0 0.0"
       rpy="0.0 0.0 0.0" />
-	<parent link="torso_head_link" />
-    <child link="torso_head_tilt_link" />
+	<parent link="head_link" />
+    <child link="head_tilt_link" />
     <!-- check -->
     <!-- axis xyz="0 1 0" / -->
@@ -301,12 +301,12 @@
     <dynamics damping="${joint_damping}" friction="${joint_friction}"/>
   </joint>
-  <transmission name="torso_head_tilt_trans">
+  <transmission name="head_tilt_trans">
 	 <type>transmission_interface/SimpleTransmission</type>
-     <joint name="torso_head_tilt_joint">
+     <joint name="head_tilt_joint">
 		<hardwareInterface>EffortJointInterface</hardwareInterface>
 	 </joint>
-     <actuator name="torso_head_tilt_motor">
-        <mechanicalReduction>${torso_head_tilt_joint_mechanical_reduction}</mechanicalReduction>
-		<motorTorqueConstant>${torso_head_tilt_joint_motor_torque_constant}</motorTorqueConstant>
+     <actuator name="head_tilt_motor">
+        <mechanicalReduction>${head_tilt_joint_mechanical_reduction}</mechanicalReduction>
+		<motorTorqueConstant>${head_tilt_joint_motor_torque_constant}</motorTorqueConstant>
 	 </actuator>
   </transmission>
