Commit message: TORSO_DESCRIPTION: Fix on URDF

File: rb1_torso_description/urdf/rb1_torso_3dof.urdf.xacro (robot description, xacro)
@@ -126,18 +126,32 @@
       <parent link="torso_link" />
       <child link="torso_slider_link" />
-      <axis xyz="0 0 1" />
-      <limit effort="${joint_effort_limit_torso}" velocity="${joint_velocity_limit_torso}" upper="${0.360}" lower="${0}"/>
+      <axis xyz="0 0 -1" />
+      <limit effort="${joint_effort_limit_torso}" velocity="${joint_velocity_limit_torso}" upper="${0}" lower="${-0.37}"/>
       <dynamics damping="${joint_damping}" friction="${joint_friction}"/>
     </joint>
     <transmission name="torso_slider_trans">
-    <type>transmission_interface/SimpleTransmission</type>
+      <type>transmission_interface/SimpleTransmission</type>
       <joint name="torso_slider_joint">
-      <hardwareInterface>hardware_interface/EffortJointInterface</hardwareInterface>
+        <hardwareInterface>hardware_interface/EffortJointInterface</hardwareInterface>
       </joint>
       <actuator name="torso_slider_motor">
-          <mechanicalReduction>${torso_slider_joint_mechanical_reduction}</mechanicalReduction>
-      <motorTorqueConstant>${torso_slider_joint_motor_torque_constant}</motorTorqueConstant>
-    </actuator>
+        <hardwareInterface>hardware_interface/EffortJointInterface</hardwareInterface>
+        <mechanicalReduction>${torso_slider_joint_mechanical_reduction}</mechanicalReduction>
+        <motorTorqueConstant>${torso_slider_joint_motor_torque_constant}</motorTorqueConstant>
+      </actuator>
     </transmission>
+    <!--joint
+      name="torso_slider_joint"
+        type="fixed">
+      <origin
+        xyz="0.07 0 0.091"
+        rpy="0.0 0.0 0.0" />
+      <parent
+        link="torso_link" />
+      <child
+        link="torso_slider_link" />
+      <axis
+        xyz="0 0 0" />
+    </joint-->
     <link name="torso_cover_link">
       <inertial>
@@ -213,13 +227,27 @@
     </joint>
     <transmission name="head_pan_trans">
-    <type>transmission_interface/SimpleTransmission</type>
-      <joint name="head_pan_joint">
+      <type>transmission_interface/SimpleTransmission</type>
+        <joint name="head_pan_joint">
+            <hardwareInterface>hardware_interface/EffortJointInterface</hardwareInterface>
+        </joint>
+        <actuator name="head_pan_motor">
           <hardwareInterface>hardware_interface/EffortJointInterface</hardwareInterface>
-      </joint>
-      <actuator name="head_pan_motor">
           <mechanicalReduction>${head_pan_joint_mechanical_reduction}</mechanicalReduction>
-      <motorTorqueConstant>${head_pan_joint_motor_torque_constant}</motorTorqueConstant>
-    </actuator>
+          <motorTorqueConstant>${head_pan_joint_motor_torque_constant}</motorTorqueConstant>
+      </actuator>
     </transmission>
+    <!--joint
+      name="head_pan_joint"
+        type="fixed">
+      <origin
+        xyz="0.055 0.0 0.621"
+        rpy="0.0 0.0 0.0" />
+      <parent
+        link="torso_slider_link" />
+      <child
+        link="head_link" />
+      <axis
+        xyz="0 0 0" />
+    </joint-->
     <link name="head_tilt_link">
       <inertial>
@@ -255,18 +283,32 @@
       <parent link="head_link" />
       <child link="head_tilt_link" />
-      <axis xyz="0 -1 0"/>
+      <axis xyz="0 1 0"/>
       <limit effort="${joint_effort_limit}" velocity="${joint_velocity_limit}" upper="${PI/4}" lower="${-PI/4}"/>
       <dynamics damping="${joint_damping}" friction="${joint_friction}"/>
     </joint>
     <transmission name="head_tilt_trans">
-    <type>transmission_interface/SimpleTransmission</type>
-      <joint name="head_tilt_joint">
-      <hardwareInterface>hardware_interface/EffortJointInterface</hardwareInterface>
-    </joint>
-      <actuator name="head_tilt_motor">
-          <mechanicalReduction>${head_tilt_joint_mechanical_reduction}</mechanicalReduction>
-      <motorTorqueConstant>${head_tilt_joint_motor_torque_constant}</motorTorqueConstant>
-    </actuator>
+      <type>transmission_interface/SimpleTransmission</type>
+        <joint name="head_tilt_joint">
+          <hardwareInterface>hardware_interface/EffortJointInterface</hardwareInterface>
+        </joint>
+        <actuator name="head_tilt_motor">
+        <hardwareInterface>hardware_interface/EffortJointInterface</hardwareInterface>
+        <mechanicalReduction>${head_tilt_joint_mechanical_reduction}</mechanicalReduction>
+        <motorTorqueConstant>${head_tilt_joint_motor_torque_constant}</motorTorqueConstant>
+      </actuator>
     </transmission>
+    <!--joint
+      name="head_tilt_joint"
+        type="fixed">
+      <origin
+        xyz="0.081 0.0 0.0"
+        rpy="0.0 0.0 0.0" />
+      <parent
+        link="head_link" />
+      <child
+        link="head_tilt_link" />
+      <axis
+        xyz="0 0 0" />
+    </joint-->
   </xacro:macro>
 </robot>

Commit message: Minor corrections

File: rb1_torso_description/urdf/rb1_torso_3dof.urdf.xacro (robot description, xacro)
@@ -126,6 +126,6 @@
       <parent link="torso_link" />
       <child link="torso_slider_link" />
-      <axis xyz="0 0 -1" />
-      <limit effort="${joint_effort_limit_torso}" velocity="${joint_velocity_limit_torso}" upper="${0}" lower="${-0.37}"/>
+      <axis xyz="0 0 1" />
+      <limit effort="${joint_effort_limit_torso}" velocity="${joint_velocity_limit_torso}" upper="${0.3645}" lower="${0}"/>
       <dynamics damping="${joint_damping}" friction="${joint_friction}"/>
     </joint>

File: rb1_torso_description/urdf/rb1_torso_std.urdf.xacro (robot description, xacro)
@@ -17,5 +17,5 @@
 		<xacro:rb1_torso_3dof base_parent="${base_parent}" hq="${hq}" />
 		<!-- RGBD sensor -->
-		<xacro:sensor_orbbec_astra prefix="head_camera" parent="head_tilt_link" prefix_topic="head_rgbd_camera">
+		<xacro:sensor_orbbec_astra prefix="rb1_torso_rgbd_camera" parent="head_tilt_link" prefix_topic="head_rgbd_camera">
 			<origin xyz="0.055 0.0125 0.028" rpy="0 0 0"/>
 		</xacro:sensor_orbbec_astra>

Commit message: Solved problem with arm planning libraries

File: rb1_torso_description/urdf/rb1_torso_3dof.urdf.xacro (robot description, xacro)
@@ -31,5 +31,5 @@
         <xacro:unless value="${hq}">
         <geometry>
-        <mesh filename="package://rb1_torso_description/meshes/torsos/rb1v2_superior1.stl"/>
+        <mesh filename="package://rb1_torso_description/meshes/torsos/rb1v2_superior1.dae"/>
         </geometry>
         </xacro:unless>
@@ -66,5 +66,5 @@
         <xacro:unless value="${hq}">
         <geometry>
-        <mesh filename="package://rb1_torso_description/meshes/torsos/rb1v2_guide.stl"/>
+        <mesh filename="package://rb1_torso_description/meshes/torsos/rb1v2_guide.dae"/>
         </geometry>
         </xacro:unless>
@@ -108,5 +108,5 @@
         <xacro:unless value="${hq}">
         <geometry>
-        <mesh filename="package://rb1_torso_description/meshes/torsos/rb1v2_superior2.stl"/>
+        <mesh filename="package://rb1_torso_description/meshes/torsos/rb1v2_superior2.dae"/>
         </geometry>
         </xacro:unless>
@@ -169,5 +169,5 @@
         <xacro:unless value="${hq}">
         <geometry>
-        <mesh filename="package://rb1_torso_description/meshes/torsos/rb1v2_rear_cover.stl"/>
+        <mesh filename="package://rb1_torso_description/meshes/torsos/rb1v2_rear_cover.dae"/>
         </geometry>
         </xacro:unless>
@@ -204,5 +204,5 @@
         <xacro:unless value="${hq}">
         <geometry>
-        <mesh filename="package://rb1_torso_description/meshes/heads/rb1v2_head1.stl"/>
+        <mesh filename="package://rb1_torso_description/meshes/heads/rb1v2_head1.dae"/>
         </geometry>
         </xacro:unless>
@@ -265,5 +265,5 @@
         <xacro:unless value="${hq}">
         <geometry>
-        <mesh filename="package://rb1_torso_description/meshes/heads/rb1v2_head2.stl"/>
+        <mesh filename="package://rb1_torso_description/meshes/heads/rb1v2_head2.dae"/>
         </geometry>
         </xacro:unless>
